File: Color Magic/s100_ColorMagic-1.1-004.kicad_sch (KiCad schematic)
At the start: 0 parts

Commit message: Add files via upload
Other:
- note added: "NOTE 2: After using an automated BOM analysis and comparing to the actual board, there are four connections on three chips that do not match the schematic. All are drawn connecting to VCC yet they are open connections on the board. U63.4 U64.4 and U64.10 U65.4 U64.10 and U65.4 are connected together. These are drawn with tie points to help with further analysis, which shows all of them can be saf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"
- note removed: "NOTE 2: After using an automated BOM analysis and comparing to the actual board, there are four connections on three chips that do not match the schematic. All are drawn connecting to VCC. They appear to be open connections. U63.4 U64.4 and U64.10 U65.4 U64.10 and U65.4 are connected together."
Changed lines of the file:
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@@
     (effects (font (size 1.27 1.27)) (justify left bottom))
   )
-  (text "NOTE 2:\n\nAfter using an automated BOM analysis and\ncomparing to the actual board, there are \nfour connections on three chips that do not\nmatch the schematic. All are drawn connecting\nto VCC. They appear to be open connections.\n\nU63.4\nU64.4 and U64.10\nU65.4\n\nU64.10 and U65.4 are connected together."
-    (at 201.93 87.884 0)
+  (text "NOTE 2:\n\nAfter using an automated BOM analysis and\ncomparing to the actual board, there are \nfour connections on three chips that do not\nmatch the schematic. All are drawn connecting\nto VCC yet they are open connections on the\nboard.\n\nU63.4\nU64.4 and U64.10\nU65.4\n\nU64.10 and U65.4 are connected together.\n\nThese are drawn with tie points to help with\nfurther analysis, which shows all of them can\nbe safely tied to Vcc."
+    (at 201.676 97.79 0)
     (effects (font (size 1.27 1.27)) (justify left bottom))
   )
-  (text "ERRATA from 1.0 to 1.1-002:\n00. v1.0 of board was trashed.\n01. Resistor footprints are one size too small -- 1/4w uses 1/8w, etc. \n	Due to space limitations, left at 1/8w.\n02. U49/78L12 silkscreen is backwards. Corrected.\n03. Several chips have unconnected VCC or GND leads that might be from\n	the use of ONE and ZERO. Corrected.\n\nERRATA from 1.1-002 to 1.1-003\n	v.003 was never manufactured.\n\nERRATA from 1.1-003 to 1.1-004\n01. J6 (address select) is flipped. Rotated 180.\n02. Design relies on SLAVE_CLR [54] for reset, but not all boards (like\n    the SCP 200B) generate that signal. Reused spare gate of the LS125\n    and added a jumper and pull-up to generate that signal driven by\n    POC [99].\n03. Changed memory chip wiring to be similar to the original, using\n    MA13 as the CS* and grounding A13 and A14 of the 62256 (thus making\n    it a 6264 albeit with only one chip select).\n04. Discovered that A6 is connected twice on U55. Changed second to\n    A5.\n"
-    (at 18.796 149.098 0)
+  (text "ERRATA from 1.0 to 1.1-002:\n00. v1.0 of board was trashed.\n01. Resistor footprints are one size too small -- 1/4w uses 1/8w, etc. \n	Due to space limitations, left at 1/8w.\n02. U49/78L12 silkscreen is backwards. Corrected.\n03. Several chips have unconnected VCC or GND leads that might be from\n	the use of ONE and ZERO. Corrected.\n\nERRATA from 1.1-002 to 1.1-003\n	v.003 was never manufactured.\n\nERRATA from 1.1-003 to 1.1-004\n01. J6 (address select) is flipped. Rotated 180.\n02. Design relies on SLAVE_CLR [54] for reset, but not all boards (like\n    the SCP 200B) generate that signal. Reused spare gate of the LS125\n    and added a jumper and pull-up to generate that signal driven by\n    POC [99].\n03. Changed memory chip wiring to be similar to the original, using\n    MA13 as the CS* and grounding A13 and A14 of the 62256 (thus making\n    it a 6264 albeit with only one chip select).\n04. Discovered that A6 is connected twice on U55. Changed second to\n    A5.\n\nThe 1.1-004 version works."
+    (at 19.304 154.432 0)
     (effects (font (size 1.27 1.27)) (justify left bottom))
   )
