File: Color Magic/buffmem.kicad_sch (KiCad schematic)
At the start: 15 parts, among them U28 74LS04, U32 74LS04, U39 74LS244, U40 74LS244, U41 74LS244, U42 74LS373, U43 74LS373, U47 74LS244, U48 74LS244, U57 74LS244, U58 74LS244, U59 74LS244, U60 74LS373, U7 HM62256BLP, U8 HM62256BLP

Commit message: Add files via upload
Connections:
- net GND: no longer U7.1 (A14), U8.1 (A14)
- new net ZERO: U7.1 (A14), U8.1 (A14)
Changed lines of the file:
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@@
   (title_block
     (title "Lomas Color Magic Redux")
-    (date "2023-03-04")
+    (date "2023-04-14")
     (rev "1.0-001")
     (company "Lomas Data Produtcs")
@@
     (comment 2 "Schematic page 1A")
   )
-  (junction (at 125.476 126.746) (diameter 0) (color 0 0 0 0)
-  )
   (junction (at 113.284 155.702) (diameter 0) (color 0 0 0 0)
-  )
-  (junction (at 125.476 68.58) (diameter 0) (color 0 0 0 0)
   )
   (no_connect (at 213.36 87.63))
@@
   (no_connect (at 101.346 191.77))
   (no_connect (at 126.746 191.77))
-  (wire (pts (xy 138.176 126.746) (xy 125.476 126.746))
-    (stroke (width 0) (type default) (color 0 0 0 0))
-  )
   (wire (pts (xy 238.76 50.292) (xy 238.76 52.832))
     (stroke (width 0) (type default) (color 0 0 0 0))
@@
   )
   (wire (pts (xy 138.176 121.666) (xy 138.176 126.746))
-    (stroke (width 0) (type default) (color 0 0 0 0))
-  )
-  (wire (pts (xy 138.176 68.58) (xy 125.476 68.58))
     (stroke (width 0) (type default) (color 0 0 0 0))
   )
@@
     (effects (font (size 1.27 1.27)) (justify left bottom))
   )
+  (label "ZERO" (at 138.176 124.714 0)
+    (effects (font (size 1.27 1.27)) (justify left bottom))
+  )
+  (label "ZERO" (at 138.176 66.294 0)
+    (effects (font (size 1.27 1.27)) (justify left bottom))
+  )

Commit message: Add files via upload
Updated to current version. Still plotting...
Parts:
- U28, U32: footprint Package_DIP:DIP-14_W7.62mm_Socket_LongPads -> Package_DIP:DIP-14_W7.62mm_Socket
- U39, U40, U41, U42, U43, U47, U48, U57, U58, U59, U60: footprint Package_DIP:DIP-20_W7.62mm_Socket_LongPads -> Package_DIP:DIP-20_W7.62mm_Socket
Connections:
- net ZERO is gone; now on net GND: U7.1 (A14), U8.1 (A14)

Commit message: Add files via upload
Parts:
- removed U32: 74LS04, Package_DIP:DIP-14_W7.62mm_Socket, symbol 74xx:74LS04
Other:
- note added: "MA14"
- note removed: "NOTE: DA12 and DA13 connect to PAL U1. Need to check the board to see if this is correct."
- moved on the sheet: U28A

Commit message: Add files via upload
Connections:
- net GND: now also U7.26 (A13), U8.26 (A13); no longer U7.20 (~{CS}), U8.20 (~{CS})
- net MA13: now also U7.20 (~{CS}), U8.20 (~{CS}); no longer U7.26 (A13), U8.26 (A13)
- net MDO0 renamed MD0
- net MDO1 renamed MD1
- net MDO10 renamed MD10
- net MDO11 renamed MD11
- net MDO12 renamed MD12
- net MDO13 renamed MD13
- net MDO14 renamed MD14
- net MDO15 renamed MD15
- net MDO2 renamed MD2
- net MDO3 renamed MD3
- net MDO4 renamed MD4
- net MDO5 renamed MD5
- net MDO6 renamed MD6
- net MDO7 renamed MD7
- net MDO8 renamed MD8
- net MDO9 renamed MD9
- no-connect marks 8 -> 9
Other:
- note added: "NOTE: Original used two stacked 6264 RAM chips in each location with MA13 connecting to /CS1 and /MA13 connecting to CS2. To select the chip, MA13 = L, driving /CS1 low. Gate 28A inverts MA13 to drive CS2 = H. A13 and A14 are held low to make the 62256 into a 6264 (albeit with one CS pin)."
- note removed: "NOTE: Original used two stacked 6264 RAM chips in each location with MA13/*MA13 acting as a select connected to /CS on each of the stacked chips."
- moved on the sheet: U28A, U39, U40, U42, U43, U58, U60
