File: Color Magic/clockaddr.kicad_sch (KiCad schematic)
At the start: 31 parts, among them U16 PAL20L10, U18 PAL16L8, U19 74LS04, U28 74LS04, U29 74LS174, U30 74LS04, U32 74LS04, U33 74LS00, U46 74ALS174, U52 74LS14, U54 74LS688, U55 PAL20L10, U56 74LS688, U61 PAL16L8, U62 74LS14, U63 74LS74, U65 74LS74, U66 74LS06, U69 74LS38, U9 74LS08, Y1 14.31818MHz

Commit message: Add files via upload
Connections:
- net GND: no longer JP12.1 (Pin_1), JP12.11 (Pin_11), JP12.3 (Pin_3), JP12.5 (Pin_5), JP12.7 (Pin_7), JP12.9 (Pin_9), JP6.10 (Pin_10), JP6.12 (Pin_12), JP6.14 (Pin_14), JP6.16 (Pin_16), JP6.2 (Pin_2), JP6.4 (Pin_4), JP6.6 (Pin_6), JP6.8 (Pin_8), U56.1 (G), U56.15 (P6), U56.16 (R6)
- net VCC: no longer RN2.1 (common), U63.4 (~{S}), U65.4 (~{S})
- new net ONE: RN2.1 (common), U63.4 (~{S}), U65.4 (~{S})
- new net ZERO: JP12.1 (Pin_1), JP12.11 (Pin_11), JP12.3 (Pin_3), JP12.5 (Pin_5), JP12.7 (Pin_7), JP12.9 (Pin_9), JP6.10 (Pin_10), JP6.12 (Pin_12), JP6.14 (Pin_14), JP6.16 (Pin_16), JP6.2 (Pin_2), JP6.4 (Pin_4), JP6.6 (Pin_6), JP6.8 (Pin_8), U56.1 (G), U56.15 (P6), U56.16 (R6)
Changed lines of the file:
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@@
   (title_block
     (title "Lomas Color Magic Redux")
-    (date "2023-03-04")
+    (date "2023-04-14")
     (rev "1.0-001")
     (company "Lomas Data Produtcs")
@@
   (junction (at 63.754 257.81) (diameter 0) (color 0 0 0 0)
   )
-  (junction (at 260.35 73.406) (diameter 0) (color 0 0 0 0)
-  )
   (junction (at 137.668 232.41) (diameter 0) (color 0 0 0 0)
   )
@@
   (junction (at 145.542 140.97) (diameter 0) (color 0 0 0 0)
   )
-  (junction (at 273.05 81.026) (diameter 0) (color 0 0 0 0)
-  )
   (junction (at 243.332 63.246) (diameter 0) (color 0 0 0 0)
   )
@@
   )
   (junction (at 63.5 83.82) (diameter 0) (color 0 0 0 0)
-  )
-  (junction (at 124.46 143.51) (diameter 0) (color 0 0 0 0)
   )
   (junction (at 153.162 125.73) (diameter 0) (color 0 0 0 0)
@@
     (stroke (width 0) (type default) (color 0 0 0 0))
   )
-  (wire (pts (xy 260.35 81.026) (xy 260.35 73.406))
-    (stroke (width 0) (type default) (color 0 0 0 0))
-  )
   (wire (pts (xy 38.862 151.638) (xy 38.862 159.258))
     (stroke (width 0) (type default) (color 0 0 0 0))
@@
     (stroke (width 0) (type default) (color 0 0 0 0))
   )
-  (wire (pts (xy 124.46 143.51) (xy 124.46 145.542))
-    (stroke (width 0) (type default) (color 0 0 0 0))
-  )
   (wire (pts (xy 137.16 135.89) (xy 155.702 135.89))
     (stroke (width 0) (type default) (color 0 0 0 0))
   )
   (wire (pts (xy 243.332 63.246) (xy 243.332 65.786))
-    (stroke (width 0) (type default) (color 0 0 0 0))
-  )
-  (wire (pts (xy 273.05 81.026) (xy 260.35 81.026))
     (stroke (width 0) (type default) (color 0 0 0 0))
   )
@@
   (text "Default:\nJP8: 1-2" (at 126.238 221.488 0)
     (effects (font (size 1.27 1.27)) (justify left bottom))
+  )
+  (label "ZERO" (at 260.35 42.926 180)
+    (effects (font (size 1.27 1.27)) (justify right bottom))
+  )
+  (label "ONE" (at 168.656 191.008 180)
+    (effects (font (size 1.27 1.27)) (justify right bottom))
+  )
+  (label "ZERO" (at 243.332 50.546 180)
+    (effects (font (size 1.27 1.27)) (justify right bottom))
+  )
+  (label "ONE" (at 155.702 165.862 180)
+    (effects (font (size 1.27 1.27)) (justify right bottom))
+  )
+  (label "ZERO" (at 124.46 125.73 180)
+    (effects (font (size 1.27 1.27)) (justify right bottom))
+  )
+  (label "ONE" (at 297.434 112.268 180)
+    (effects (font (size 1.27 1.27)) (justify right bottom))
   )
   (global_label "A15" (shape input) (at 159.512 120.65 180) (fields_autoplaced)
@@
     (pin "1")
   )
-  (symbol (lib_id "power:GND") (at 260.35 42.926 270) (unit 1)
-    (in_bom yes) (on_board yes)
-    (property "Reference" "#PWR0518" (id 0) (at 254 42.926 0)
-      (effects (font (size 1.27 1.27)) hide)
-    )
-    (property "Value" "GND" (id 1) (at 253.492 43.18 90)
-      (effects (font (size 1.27 1.27)) (justify left))
-    )
-    (property "Footprint" "" (id 2) (at 260.35 42.926 0)
-      (effects (font (size 1.27 1.27)) hide)
-    )
-    (property "Datasheet" "" (id 3) (at 260.35 42.926 0)
-      (effects (font (size 1.27 1.27)) hide)
-    )
-    (pin "1")
-  )
   (symbol (lib_id "74xx:74LS00") (at 142.24 196.088 0) (unit 2)
     (in_bom yes) (on_board yes) (fields_autoplaced)
@@
     (pin "7")
   )
-  (symbol (lib_id "power:VCC") (at 155.702 165.862 180) (unit 1)
-    (in_bom yes) (on_board yes) (fields_autoplaced)
-    (property "Reference" "#PWR0511" (id 0) (at 155.702 162.052 0)
-      (effects (font (size 1.27 1.27)) hide)
-    )
-    (property "Value" "VCC" (id 1) (at 157.099 167.5658 0)
-      (effects (font (size 1.27 1.27)) (justify right))
-    )
-    (property "Footprint" "" (id 2) (at 155.702 165.862 0)
-      (effects (font (size 1.27 1.27)) hide)
-    )
-    (property "Datasheet" "" (id 3) (at 155.702 165.862 0)
-      (effects (font (size 1.27 1.27)) hide)
-    )
-    (pin "1")
-  )
   (symbol (lib_id "74xx:74LS08") (at 333.756 228.6 0) (unit 4)
     (in_bom yes) (on_board yes) (fields_autoplaced)
@@
     (pin "14")
     (pin "7")
-  )
-  (symbol (lib_id "power:GND") (at 124.46 145.542 0) (unit 1)
-    (in_bom yes) (on_board yes) (fields_autoplaced)
-    (property "Reference" "#PWR0509" (id 0) (at 124.46 151.892 0)
-      (effects (font (size 1.27 1.27)) hide)
-    )
-    (property "Value" "GND" (id 1) (at 124.46 149.9854 0))
-    (property "Footprint" "" (id 2) (at 124.46 145.542 0)
-      (effects (font (size 1.27 1.27)) hide)
-    )
-    (property "Datasheet" "" (id 3) (at 124.46 145.542 0)
-      (effects (font (size 1.27 1.27)) hide)
-    )
-    (pin "1")
   )
   (symbol (lib_id "74xx:74LS74") (at 297.434 119.888 0) (unit 1)
@@
     (pin "7")
   )
-  (symbol (lib_id "power:VCC") (at 297.434 112.268 0) (unit 1)
-    (in_bom yes) (on_board yes) (fields_autoplaced)
-    (property "Reference" "#PWR0521" (id 0) (at 297.434 116.078 0)
-      (effects (font (size 1.27 1.27)) hide)
-    )
-    (property "Value" "VCC" (id 1) (at 297.434 108.6922 0))
-    (property "Footprint" "" (id 2) (at 297.434 112.268 0)
-      (effects (font (size 1.27 1.27)) hide)
-    )
-    (property "Datasheet" "" (id 3) (at 297.434 112.268 0)
-      (effects (font (size 1.27 1.27)) hide)
-    )
-    (pin "1")
-  )
   (symbol (lib_id "power:VCC") (at 227.076 163.068 0) (unit 1)
     (in_bom yes) (on_board yes)
@@
     (pin "7")
   )
-  (symbol (lib_id "power:VCC") (at 168.656 191.008 0) (unit 1)
-    (in_bom yes) (on_board yes)
-    (property "Reference" "#PWR0510" (id 0) (at 168.656 194.818 0)
-      (effects (font (size 1.27 1.27)) hide)
-    )
-    (property "Value" "VCC" (id 1) (at 166.878 187.452 0)
-      (effects (font (size 1.27 1.27)) (justify left))
-    )
-    (property "Footprint" "" (id 2) (at 168.656 191.008 0)
-      (effects (font (size 1.27 1.27)) hide)
-    )
-    (property "Datasheet" "" (id 3) (at 168.656 191.008 0)
-      (effects (font (size 1.27 1.27)) hide)
-    )
-    (pin "1")
-  )
   (symbol (lib_id "74xx:74LS174") (at 43.18 91.44 0) (unit 1)

Commit message: Add files via upload
Updated to current version. Still plotting...
Parts:
- R7, R8: footprint Resistor_THT:R_Axial_DIN0204_L3.6mm_D1.6mm_P5.08mm_Horizontal -> Resistor_THT:R_Axial_DIN0207_L6.3mm_D2.5mm_P7.62mm_Horizontal
- U16, U55: footprint Package_DIP:DIP-24_W7.62mm_Socket_LongPads -> Package_DIP:DIP-24_W7.62mm_Socket
- U18, U54, U56, U61: footprint Package_DIP:DIP-20_W7.62mm_Socket_LongPads -> Package_DIP:DIP-20_W7.62mm_Socket
- U19, U28, U30, U32, U33, U52, U62, U63, U65, U66, U69, U9: footprint Package_DIP:DIP-14_W7.62mm_Socket_LongPads -> Package_DIP:DIP-14_W7.62mm_Socket
- U29, U46: footprint Package_DIP:DIP-16_W7.62mm_Socket_LongPads -> Package_DIP:DIP-16_W7.62mm_Socket
Connections:
- net ONE is gone; now on net VCC: RN2.1 (common), U63.4 (~{S}), U65.4 (~{S})
- net ZERO is gone; now on net GND: JP12.1 (Pin_1), JP12.11 (Pin_11), JP12.3 (Pin_3), JP12.5 (Pin_5), JP12.7 (Pin_7), JP12.9 (Pin_9), JP6.10 (Pin_10), JP6.12 (Pin_12), JP6.14 (Pin_14), JP6.16 (Pin_16), JP6.2 (Pin_2), JP6.4 (Pin_4), JP6.6 (Pin_6), JP6.8 (Pin_8), U56.1 (G), U56.15 (P6), U56.16 (R6)
Other:
- note added: "NOTE: On schematic, pin 17 is "HLCK" so possibly typo."
- note removed: "NOTE: Check pin 9 against others."

Commit message: Add files via upload
Parts:
- added unit 4 of U32
- U66: value 74LS06 -> 7406
Connections:
- net GND: now also JP12.10 (Pin_10), JP12.12 (Pin_12), JP12.2 (Pin_2), JP12.4 (Pin_4), JP12.6 (Pin_6), JP12.8 (Pin_8); no longer JP12.1 (Pin_1), JP12.11 (Pin_11), JP12.3 (Pin_3), JP12.5 (Pin_5), JP12.7 (Pin_7), JP12.9 (Pin_9)
- net HCLK: now also U32.9
- net /HCLK: now also U32.8
- net at U56.12 (R4): now also JP12.9 (Pin_9); no longer JP12.10 (Pin_10)
- net at U56.14 (R5): now also JP12.11 (Pin_11); no longer JP12.12 (Pin_12)
- net at U56.3 (R0): now also JP12.1 (Pin_1); no longer JP12.2 (Pin_2)
- net at U56.5 (R1): now also JP12.3 (Pin_3); no longer JP12.4 (Pin_4)
- net at U56.7 (R2): now also JP12.5 (Pin_5); no longer JP12.6 (Pin_6)
- net at U56.9 (R3): now also JP12.7 (Pin_7); no longer JP12.8 (Pin_8)
- no-connect marks 28 -> 26
Other:
- note added: "Default (L->R) 0-0-0--1-0-1-1--1 ------{-- B --}{8} [0x0B800]"
- note added: "Default: JP7: 2-3"
- note added: "NOTE: Board uses 7406; LS family seems to work fine."
- note added: "NOTE: Hanging line on pSYNC"
- note added: "NOTE: Possibly replace all with TTL oscillator."
- note added: "NOTE: R7/R8 was specified as 1.0k on schematic but the board I looked at had 470Q. On the reproduction, 1.0k works better. Also, install a jumper in place of C8. This should result in a frequency of ~14.305MHz."
- note removed: "Default (L->R) 0-0-0-1-0-1-1-1"
- note removed: "Default: JP7: 1-2"
- note removed: "NOTE: On schematic, pin 17 is "HLCK" so possibly typo."
- note removed: "NOTE: R7/R8 was 1.0k on schematic."
- moved on the sheet: C8, JP6, JP7, JP8, JP9, R7, R8, RN2, U28B, U28D, U28E, U28F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

Commit message: Add files via upload
Parts:
- removed C8: 10pF, Capacitor_THT:C_Disc_D4.3mm_W1.9mm_P5.00mm, symbol Device:C
- removed R7, R8: 470Q, Resistor_THT:R_Axial_DIN0207_L6.3mm_D2.5mm_P7.62mm_Horizontal, symbol Device:R
- removed Y1: 14.31818MHz, Crystal:Crystal_HC49-U_Horizontal, symbol Device:Crystal_Small
- added TP1, TP3, TP4: TestPoint, TestPoint:TestPoint_THTPad_1.0x1.0mm_Drill0.5mm, symbol Connector:TestPoint
- added X1: 14.31818MHz, Oscillator:Oscillator_DIP-14, symbol Oscillator:CXO_DIP14
- U16, U55: symbol RAC_Custom2:PAL20L10 -> RAC_Custom:PAL20L10
Connections:
- net 14MCLK: now also TP1.1, X1.8 (OUT); no longer U28.10
- net A6: no longer U55.8 (I8)
- net GND: now also X1.7 (GND)
- net VCC: now also X1.14 (Vcc); no longer U63.4 (~{S}), U65.4 (~{S})
- net at U28.12: no longer U28.11
- net at U28.4: no longer U28.13
- net IDSELECT: no longer names the net of U55.1 (I1), U56.19 (P=R)
- net SYNC_SRC: no longer names the net of U62.12, U65.3 (C)
- new net: TP3.1, U63.4 (~{S})
- new net A5: U55.8 (I8)
- new net U65.4: TP4.1, U65.4 (~{S})
- no-connect marks 26 -> 35
Other:
- note added: "Board Select"
- note added: "Default: All Closed 0000-00xx-xxxx-xxxx 03xx"
- note added: "NOTE: On the prototype U63.4 is left floating. In the IBM CGA adapter, it's tied to Vcc."
- note added: "NOTE: On the prototype U65.4 is connected to U64.10."
- note added: "NOTE: R7/R8 was specified as 1.0kQ on schematic but 470Q was used in the actual manufacturing of the board. Prior to converting to a TTL oscillator, 1.0kQ was determined to work better. Also, install a jumper in place of C8. This should result in a frequency of ~14.305MHz."
- note added: "NOTE: The original circuit consisted of a crystal-based frequency generator using 3 gates from U28, a parallel capacitor and two resistors."
- note removed: "Default: All Closed"
- note removed: "NOTE: Hanging line on pSYNC"
- note removed: "NOTE: Possibly replace all with TTL oscillator."
- note removed: "NOTE: R7/R8 was specified as 1.0k on schematic but the board I looked at had 470Q. On the reproduction, 1.0k works better. Also, install a jumper in place of C8. This should result in a frequency of ~14.305MHz."
- moved on the sheet: JP15, JP6, JP7, JP9, RN2, U28B, U28D, U28E, U28F, U30A, U30C, U32A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

Commit message: Add files via upload
Other:
- note added: "TP3: On the prototype U63.4 is left floating. In the IBM CGA adapter, it's tied to Vcc. TIE TO VCC"
- note added: "TP4: On the prototype U65.4 is connected to U64.10. TIE TO VCC."
- note removed: "NOTE: On the prototype U63.4 is left floating. In the IBM CGA adapter, it's tied to Vcc."
- note removed: "NOTE: On the prototype U65.4 is connected to U64.10."
Changed lines of the file:
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@@
     (effects (font (size 1.27 1.27)) (justify left bottom))
   )
-  (text "NOTE: On the prototype U63.4 is left floating.\nIn the IBM CGA adapter, it's tied to Vcc."
-    (at 207.264 206.248 0)
+  (text "TP3: On the prototype U63.4 is left floating.\nIn the IBM CGA adapter, it's tied to Vcc.\n\nTIE TO VCC"
+    (at 208.026 211.328 0)
     (effects (font (size 1.27 1.27)) (justify left bottom))
   )
@@
     (effects (font (size 1.27 1.27)) (justify left bottom))
   )
-  (text "NOTE: On the prototype U65.4 is connected\nto U64.10."
-    (at 237.744 156.21 0)
+  (text "TP4: On the prototype U65.4 is connected\nto U64.10. TIE TO VCC."
+    (at 229.87 156.718 0)
     (effects (font (size 1.27 1.27)) (justify left bottom))
   )

Commit message: Add files via upload
Final versions uploaded.
Parts:
- removed TP3, TP4: TestPoint, TestPoint:TestPoint_THTPad_1.0x1.0mm_Drill0.5mm, symbol Connector:TestPoint
Connections:
- net U65.4 is gone; now on net VCC: U65.4 (~{S})
- net VCC: now also U63.4 (~{S})
Changed lines of the file:
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@@
   (title_block
     (title "Lomas Color Magic Redux")
-    (date "2024-08-16")
-    (rev "1.1-004")
+    (date "2024-09-24")
+    (rev "1.1-005")
     (company "Lomas Data Produtcs")
     (comment 1 "Redraw/modifications (c) Richard A. Cini")
@@
   (junction (at 125.984 217.424) (diameter 0) (color 0 0 0 0)
   )
-  (junction (at 289.306 158.496) (diameter 0) (color 0 0 0 0)
-  )
   (junction (at 38.1 137.16) (diameter 0) (color 0 0 0 0)
   )
@@
     (stroke (width 0) (type default) (color 0 0 0 0))
   )
-  (wire (pts (xy 292.354 158.496) (xy 289.306 158.496))
-    (stroke (width 0) (type default) (color 0 0 0 0))
-  )
   (wire (pts (xy 242.824 83.312) (xy 242.824 68.326))
     (stroke (width 0) (type default) (color 0 0 0 0))
@@
     (stroke (width 0) (type default) (color 0 0 0 0))
   )
-  (wire (pts (xy 289.306 158.496) (xy 289.306 164.338))
-    (stroke (width 0) (type default) (color 0 0 0 0))
-  )
   (wire (pts (xy 289.306 186.182) (xy 289.306 190.246))
     (stroke (width 0) (type default) (color 0 0 0 0))
@@
     )
   )
-  (global_label "U65.4" (shape output) (at 292.354 158.496 0) (fields_autoplaced)
-    (effects (font (size 1.27 1.27)) (justify left))
-    (property "Intersheet References" "${INTERSHEET_REFS}" (id 0) (at 300.242 158.4166 0)
-      (effects (font (size 1.27 1.27)) (justify left) hide)
-    )
-  )
   (global_label "{slash}LPEN_CLR" (shape output) (at 338.582 42.926 0) (fields_autoplaced)
     (effects (font (size 1.27 1.27)) (justify left))
@@
     (pin "7")
   )
-  (symbol (lib_id "Connector:TestPoint") (at 194.056 193.04 0) (mirror y) (unit 1)
-    (in_bom yes) (on_board yes)
-    (property "Reference" "TP3" (id 0) (at 188.214 189.484 0)
-      (effects (font (size 1.27 1.27)) (justify right))
-    )
-    (property "Value" "TestPoint" (id 1) (at 184.404 191.516 0)
-      (effects (font (size 1.27 1.27)) (justify right))
-    )
-    (property "Footprint" "TestPoint:TestPoint_THTPad_1.0x1.0mm_Drill0.5mm" (id 2) (at 188.976 193.04 0)
-      (effects (font (size 1.27 1.27)) hide)
-    )
-    (property "Datasheet" "~" (id 3) (at 188.976 193.04 0)
-      (effects (font (size 1.27 1.27)) hide)
-    )
-    (pin "1")
-  )
   (symbol (lib_id "74xx:74LS04") (at 389.636 83.058 0) (unit 4)
     (in_bom yes) (on_board yes) (fields_autoplaced)
@@
     (pin "7")
   )
+  (symbol (lib_id "power:VCC") (at 194.056 193.04 0) (unit 1)
+    (in_bom yes) (on_board yes)
+    (property "Reference" "#PWR038" (id 0) (at 194.056 196.85 0)
+      (effects (font (size 1.27 1.27)) hide)
+    )
+    (property "Value" "VCC" (id 1) (at 188.214 192.278 0)
+      (effects (font (size 1.27 1.27)) (justify left))
+    )
+    (property "Footprint" "" (id 2) (at 194.056 193.04 0)
+      (effects (font (size 1.27 1.27)) hide)
+    )
+    (property "Datasheet" "" (id 3) (at 194.056 193.04 0)
+      (effects (font (size 1.27 1.27)) hide)
+    )
+    (pin "1")
+  )
   (symbol (lib_id "Device:R_Network08") (at 169.926 162.052 180) (unit 1)
     (in_bom yes) (on_board yes) (fields_autoplaced)
@@
     (pin "1")
   )
+  (symbol (lib_id "power:VCC") (at 289.306 164.338 0) (unit 1)
+    (in_bom yes) (on_board yes)
+    (property "Reference" "#PWR039" (id 0) (at 289.306 168.148 0)
+      (effects (font (size 1.27 1.27)) hide)
+    )
+    (property "Value" "VCC" (id 1) (at 283.464 163.576 0)
+      (effects (font (size 1.27 1.27)) (justify left))
+    )
+    (property "Footprint" "" (id 2) (at 289.306 164.338 0)
+      (effects (font (size 1.27 1.27)) hide)
+    )
+    (property "Datasheet" "" (id 3) (at 289.306 164.338 0)
+      (effects (font (size 1.27 1.27)) hide)
+    )
+    (pin "1")
+  )
   (symbol (lib_id "74xx:74LS04") (at 379.73 229.616 0) (unit 5)
     (in_bom yes) (on_board yes) (fields_autoplaced)
@@
     (pin "7")
   )
-  (symbol (lib_id "Connector:TestPoint") (at 289.306 158.496 0) (mirror y) (unit 1)
-    (in_bom yes) (on_board yes)
-    (property "Reference" "TP4" (id 0) (at 283.464 154.94 0)
-      (effects (font (size 1.27 1.27)) (justify right))
-    )
-    (property "Value" "TestPoint" (id 1) (at 279.654 156.972 0)
-      (effects (font (size 1.27 1.27)) (justify right))
-    )
-    (property "Footprint" "TestPoint:TestPoint_THTPad_1.0x1.0mm_Drill0.5mm" (id 2) (at 284.226 158.496 0)
-      (effects (font (size 1.27 1.27)) hide)
-    )
-    (property "Datasheet" "~" (id 3) (at 284.226 158.496 0)
-      (effects (font (size 1.27 1.27)) hide)
-    )
-    (pin "1")
-  )
   (symbol (lib_id "power:VCC") (at 272.796 100.838 0) (unit 1)
