File: Color Magic/inout.kicad_sch (KiCad schematic)
At the start: 25 parts, among them J3 Keyboard, J4 LPEN, U25 82C55A, U28 74LS04, U37 74LS322, U51 74LS125, U52 74LS14, U53 74LS74, U62 74LS14, U64 74LS74, U66 74LS06, U67 74LS92, U68 8253, U69 74LS38

Commit message: Add files via upload
Connections:
- net GND: no longer U67.6 (R0(1)), U67.7 (R0(2))
- net VCC: no longer U37.18 (SE), U37.19 (DS), U37.2 (S/P), U37.3 (D0), U53.10 (~{S}), U64.10 (~{S}), U64.4 (~{S}), U68.11 (G0), U68.14 (G1)
- new net ONE: U53.10 (~{S}), U64.10 (~{S}), U64.4 (~{S}), U68.11 (G0), U68.14 (G1)
- new net ZERO: U37.18 (SE), U37.19 (DS), U37.2 (S/P), U37.3 (D0), U67.6 (R0(1)), U67.7 (R0(2))
Changed lines of the file:
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@@
   (title_block
     (title "Lomas Color Magic Redux")
-    (date "2023-03-04")
+    (date "2023-04-14")
     (rev "1.0-001")
     (company "Lomas Data Produtcs")
@@
   (junction (at 239.522 77.724) (diameter 0) (color 0 0 0 0)
   )
-  (junction (at 174.752 105.41) (diameter 0) (color 0 0 0 0)
-  )
   (junction (at 239.522 70.104) (diameter 0) (color 0 0 0 0)
   )
@@
   (junction (at 70.104 192.786) (diameter 0) (color 0 0 0 0)
   )
-  (junction (at 116.078 66.802) (diameter 0) (color 0 0 0 0)
-  )
   (junction (at 117.856 210.566) (diameter 0) (color 0 0 0 0)
   )
-  (junction (at 44.704 146.558) (diameter 0) (color 0 0 0 0)
-  )
   (junction (at 128.778 54.102) (diameter 0) (color 0 0 0 0)
   )
@@
   (junction (at 228.092 95.25) (diameter 0) (color 0 0 0 0)
   )
-  (junction (at 57.404 156.718) (diameter 0) (color 0 0 0 0)
-  )
   (junction (at 164.338 124.968) (diameter 0) (color 0 0 0 0)
   )
@@
   )
   (junction (at 258.572 133.35) (diameter 0) (color 0 0 0 0)
-  )
-  (junction (at 128.778 59.182) (diameter 0) (color 0 0 0 0)
   )
   (junction (at 170.434 50.292) (diameter 0) (color 0 0 0 0)
@@
     (stroke (width 0) (type default) (color 0 0 0 0))
   )
-  (wire (pts (xy 44.704 146.558) (xy 44.704 156.718))
-    (stroke (width 0) (type default) (color 0 0 0 0))
-  )
   (wire (pts (xy 221.742 26.416) (xy 221.742 40.132))
     (stroke (width 0) (type default) (color 0 0 0 0))
@@
     (stroke (width 0) (type default) (color 0 0 0 0))
   )
-  (wire (pts (xy 128.778 66.802) (xy 128.778 59.182))
-    (stroke (width 0) (type default) (color 0 0 0 0))
-  )
   (wire (pts (xy 221.742 40.132) (xy 224.282 40.132))
     (stroke (width 0) (type default) (color 0 0 0 0))
@@
     (stroke (width 0) (type default) (color 0 0 0 0))
   )
-  (wire (pts (xy 116.078 66.802) (xy 128.778 66.802))
-    (stroke (width 0) (type default) (color 0 0 0 0))
-  )
   (wire (pts (xy 254.254 36.576) (xy 275.082 36.576))
     (stroke (width 0) (type default) (color 0 0 0 0))
@@
     (stroke (width 0) (type default) (color 0 0 0 0))
   )
-  (wire (pts (xy 57.404 156.718) (xy 44.704 156.718))
-    (stroke (width 0) (type default) (color 0 0 0 0))
-  )
   (wire (pts (xy 75.184 59.182) (xy 103.378 59.182))
     (stroke (width 0) (type default) (color 0 0 0 0))
@@
   )
   (wire (pts (xy 225.298 45.212) (xy 225.298 63.754))
-    (stroke (width 0) (type default) (color 0 0 0 0))
-  )
-  (wire (pts (xy 174.752 102.362) (xy 174.752 105.41))
     (stroke (width 0) (type default) (color 0 0 0 0))
   )
@@
   )
   (label "KBD_INT*" (at 256.032 36.576 0)
+    (effects (font (size 1.27 1.27)) (justify left bottom))
+  )
+  (label "ONE" (at 174.752 105.41 180)
+    (effects (font (size 1.27 1.27)) (justify right bottom))
+  )
+  (label "ZERO" (at 131.064 54.102 0)
+    (effects (font (size 1.27 1.27)) (justify left bottom))
+  )
+  (label "ONE" (at 67.31 195.326 0)
+    (effects (font (size 1.27 1.27)) (justify left bottom))
+  )
+  (label "ZERO" (at 44.704 144.018 180)
+    (effects (font (size 1.27 1.27)) (justify right bottom))
+  )
+  (label "ONE" (at 211.582 35.052 180)
+    (effects (font (size 1.27 1.27)) (justify right bottom))
+  )
+  (label "ONE" (at 67.31 182.626 0)
     (effects (font (size 1.27 1.27)) (justify left bottom))
   )
@@
     (pin "2")
   )
-  (symbol (lib_id "power:VCC") (at 174.752 102.362 0) (unit 1)
-    (in_bom yes) (on_board yes) (fields_autoplaced)
-    (property "Reference" "#PWR0715" (id 0) (at 174.752 106.172 0)
-      (effects (font (size 1.27 1.27)) hide)
-    )
-    (property "Value" "VCC" (id 1) (at 176.149 101.5258 0)
-      (effects (font (size 1.27 1.27)) (justify left))
-    )
-    (property "Footprint" "" (id 2) (at 174.752 102.362 0)
-      (effects (font (size 1.27 1.27)) hide)
-    )
-    (property "Datasheet" "" (id 3) (at 174.752 102.362 0)
-      (effects (font (size 1.27 1.27)) hide)
-    )
-    (pin "1")
-  )
   (symbol (lib_id "74xx:74LS125") (at 73.152 246.634 0) (unit 5)
     (in_bom yes) (on_board yes) (fields_autoplaced)
@@
     (pin "7")
   )
-  (symbol (lib_id "power:VCC") (at 67.31 195.326 270) (unit 1)
-    (in_bom yes) (on_board yes) (fields_autoplaced)
-    (property "Reference" "#PWR0710" (id 0) (at 63.5 195.326 0)
-      (effects (font (size 1.27 1.27)) hide)
-    )
-    (property "Value" "VCC" (id 1) (at 70.485 195.7598 90)
-      (effects (font (size 1.27 1.27)) (justify left))
-    )
-    (property "Footprint" "" (id 2) (at 67.31 195.326 0)
-      (effects (font (size 1.27 1.27)) hide)
-    )
-    (property "Datasheet" "" (id 3) (at 67.31 195.326 0)
-      (effects (font (size 1.27 1.27)) hide)
-    )
-    (pin "1")
-  )
   (symbol (lib_id "74xx:74LS125") (at 193.802 233.934 0) (unit 1)
     (in_bom yes) (on_board yes) (fields_autoplaced)
@@
     )
     (property "Datasheet" "" (id 3) (at 276.606 168.402 0)
-      (effects (font (size 1.27 1.27)) hide)
-    )
-    (pin "1")
-  )
-  (symbol (lib_id "power:VCC") (at 67.31 182.626 270) (unit 1)
-    (in_bom yes) (on_board yes) (fields_autoplaced)
-    (property "Reference" "#PWR0709" (id 0) (at 63.5 182.626 0)
-      (effects (font (size 1.27 1.27)) hide)
-    )
-    (property "Value" "VCC" (id 1) (at 70.485 183.0598 90)
-      (effects (font (size 1.27 1.27)) (justify left))
-    )
-    (property "Footprint" "" (id 2) (at 67.31 182.626 0)
-      (effects (font (size 1.27 1.27)) hide)
-    )
-    (property "Datasheet" "" (id 3) (at 67.31 182.626 0)
       (effects (font (size 1.27 1.27)) hide)
     )
@@
     (pin "9")
   )
-  (symbol (lib_id "power:VCC") (at 211.582 35.052 0) (unit 1)
-    (in_bom yes) (on_board yes)
-    (property "Reference" "#PWR0716" (id 0) (at 211.582 38.862 0)
-      (effects (font (size 1.27 1.27)) hide)
-    )
-    (property "Value" "VCC" (id 1) (at 209.55 31.496 0)
-      (effects (font (size 1.27 1.27)) (justify left))
-    )
-    (property "Footprint" "" (id 2) (at 211.582 35.052 0)
-      (effects (font (size 1.27 1.27)) hide)
-    )
-    (property "Datasheet" "" (id 3) (at 211.582 35.052 0)
-      (effects (font (size 1.27 1.27)) hide)
-    )
-    (pin "1")
-  )
   (symbol (lib_id "74xx:74LS06") (at 231.902 40.132 0) (unit 2)

Commit message: Add files via upload
Updated to current version. Still plotting...
Parts:
- R14, R16: footprint Resistor_THT:R_Axial_DIN0204_L3.6mm_D1.6mm_P5.08mm_Horizontal -> Resistor_THT:R_Axial_DIN0207_L6.3mm_D2.5mm_P7.62mm_Horizontal
- R21: footprint Resistor_THT:R_Axial_DIN0207_L6.3mm_D2.5mm_P7.62mm_Horizontal -> Resistor_THT:R_Axial_DIN0411_L9.9mm_D3.6mm_P12.70mm_Horizontal
- U28, U51, U52, U53, U62, U64, U66, U67, U69: footprint Package_DIP:DIP-14_W7.62mm_Socket_LongPads -> Package_DIP:DIP-14_W7.62mm_Socket
- U37: footprint Package_DIP:DIP-20_W7.62mm_Socket_LongPads -> Package_DIP:DIP-20_W7.62mm_Socket
Connections:
- net ONE is gone; now on net VCC: U53.10 (~{S}), U64.10 (~{S}), U64.4 (~{S}), U68.11 (G0), U68.14 (G1)
- net GND: now also U67.6 (R0(1)), U67.7 (R0(2))
- net KBD_DATA: now also C19.1, R14.1, U51.11
- net VCC: now also U37.18 (SE), U37.19 (DS), U37.2 (S/P), U37.3 (D0), U67.5 (VCC)
- net CGRDM11 renamed CGROM11
- net CGRDM12 renamed CGROM12
- removed net ZERO: U37.18 (SE), U37.19 (DS), U37.2 (S/P), U37.3 (D0), U67.6 (R0(1)), U67.7 (R0(2))
Other:
- moved on the sheet: C19, C2, C30, C37, J3, JP14, R16

Commit message: Add files via upload
Parts:
- removed JP13: CLK, Connector_PinHeader_2.54mm:PinHeader_1x03_P2.54mm_Vertical, symbol Connector_Generic:Conn_01x03
- added JP13: CLK Src, Connector_PinHeader_2.54mm:PinHeader_1x03_P2.54mm_Vertical, symbol Jumper:Jumper_3_Open
- added JP402: Jumper_2_Open, Connector_PinHeader_2.54mm:PinHeader_1x02_P2.54mm_Vertical, symbol Jumper:Jumper_2_Open
- added R401: 1.0kQ, Resistor_THT:R_Axial_DIN0207_L6.3mm_D2.5mm_P7.62mm_Horizontal, symbol Device:R
- U51: value 74LS125 -> 74125
- U66: value 74LS06 -> 7406
Connections:
- net GND: now also U51.2
- net VCC: now also R401.2
- net POC*: now reaches U51.1
- net at U51.3: now also JP402.1 (A), R401.1
- net at U68.13 (OUT1): now also JP13.3 (B)
- net at U67.8 (Q3), U68.15 (CLK1), U68.18 (CLK2): now also JP13.1 (A)
- net at U68.9 (CLK0): now also JP13.2 (C)
- new net /SLAVE_CLR: JP402.2 (B)
- no-connect marks 19 -> 16
Other:
- note added: "/DIV 8"
- note added: "NOTE: Board uses a 74125; LS family seems to work."
- note added: "SLAVE_CLR Enable: Some CPU cards do not generate SLAVE_CLR (like the SCP 200B) so this creates the same signal for the bus. Jumper only if no other card provides this signal."
- moved on the sheet: U51A

Commit message: Add files via upload
Parts:
- removed R401: 1.0kQ, Resistor_THT:R_Axial_DIN0207_L6.3mm_D2.5mm_P7.62mm_Horizontal, symbol Device:R
- removed U67: 74LS92, Package_DIP:DIP-14_W7.62mm_Socket, symbol 74xx:74LS92
- added TP5: TestPoint, TestPoint:TestPoint_THTPad_1.0x1.0mm_Drill0.5mm, symbol Connector:TestPoint
- added U67: 74LS92, Package_DIP:DIP-14_W7.62mm_Socket, symbol 74xx_IEEE:7492
Connections:
- net 14MCLK: now also U67.14 (~{CP0})
- net GND: now also U67.10 (GND), U67.6 (R0(1)), U67.7 (R0(2))
- net VCC: now also U67.5 (VCC); no longer U64.10 (~{S}), U64.4 (~{S})
- net at JP13.1 (A), U68.15 (CLK1), U68.18 (CLK2): now also U67.8 (Q3)
- net PU_RN1_8: now reaches JP402.1 (A), U51.3
- net U25.13 renamed PC4
- net U25.24 renamed PB6
- net U25.25 renamed PB7
- new net: TP5.1, U64.4 (~{S})
- new net: U67.1 (CP1), U67.12 (Q0)
- new net U65.4: U64.10 (~{S})
Other:
- note added: "NOTE: JP13 is oriented PIN 1 down."
- note added: "NOTE: On the prototype, U64.10 is connected to U65.4."
- note added: "Pull-up = 4.7k"
- moved on the sheet: C2, C30, C31, C37, J3, J4, JP10, JP402, R14, R16, U51A, U51B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

Commit message: Add files via upload
Other:
- note added: "TP5: On the prototype, U64.10 is connected to U65.4. TIE TO VCC."
- note removed: "NOTE: On the prototype, U64.10 is connected to U65.4."
Changed lines of the file:
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@@
     )
   )
-  (text "NOTE: On the prototype, U64.10 is connected to \nU65.4."
-    (at 222.25 121.412 0)
+  (text "TP5: On the prototype, U64.10 is connected to \nU65.4. TIE TO VCC."
+    (at 188.214 146.05 0)
     (effects (font (size 1.27 1.27)) (justify left bottom))
   )
@@
     )
   )
-  (global_label "SPKR_GATE" (shape output) (at 67.31 208.026 0) (fields_autoplaced)
+  (global_label "SPKR_GATE" (shape input) (at 67.31 208.026 0) (fields_autoplaced)
     (effects (font (size 1.27 1.27)) (justify left))
     (property "Intersheet References" "${INTERSHEET_REFS}" (id 0) (at 80.0966 207.9466 0)

Commit message: Add files via upload
Final versions uploaded.
Parts:
- removed TP5: TestPoint, TestPoint:TestPoint_THTPad_1.0x1.0mm_Drill0.5mm, symbol Connector:TestPoint
Connections:
- net U65.4 is gone; now on net VCC: U64.10 (~{S})
- net VCC: now also U64.4 (~{S})
Changed lines of the file:
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@@
   (title_block
     (title "Lomas Color Magic Redux")
-    (date "2024-08-16")
-    (rev "1.1-004")
+    (date "2024-09-24")
+    (rev "1.1-005")
     (company "Lomas Data Produtcs")
     (comment 1 "Redraw/modifications (c) Richard A. Cini")
@@
     (stroke (width 0) (type default) (color 0 0 0 0))
   )
-  (wire (pts (xy 204.724 115.824) (xy 207.518 115.824))
-    (stroke (width 0) (type default) (color 0 0 0 0))
-  )
   (wire (pts (xy 117.602 175.26) (xy 117.602 180.34))
     (stroke (width 0) (type default) (color 0 0 0 0))
@@
   )
   (wire (pts (xy 239.522 70.104) (xy 239.522 70.866))
-    (stroke (width 0) (type default) (color 0 0 0 0))
-  )
-  (wire (pts (xy 207.518 115.824) (xy 207.518 116.84))
     (stroke (width 0) (type default) (color 0 0 0 0))
   )
@@
   )
   (text "TP5: On the prototype, U64.10 is connected to \nU65.4. TIE TO VCC."
-    (at 188.214 146.05 0)
+    (at 182.88 145.542 0)
     (effects (font (size 1.27 1.27)) (justify left bottom))
   )
@@
     (effects (font (size 1.27 1.27)) (justify right))
     (property "Intersheet References" "${INTERSHEET_REFS}" (id 0) (at 33.4293 51.4826 0)
-      (effects (font (size 1.27 1.27)) (justify right) hide)
-    )
-  )
-  (global_label "U65.4" (shape input) (at 204.724 115.824 180) (fields_autoplaced)
-    (effects (font (size 1.27 1.27)) (justify right))
-    (property "Intersheet References" "${INTERSHEET_REFS}" (id 0) (at 196.836 115.7446 0)
       (effects (font (size 1.27 1.27)) (justify right) hide)
     )
@@
     (pin "1")
   )
+  (symbol (lib_id "power:VCC") (at 207.518 116.84 0) (unit 1)
+    (in_bom yes) (on_board yes)
+    (property "Reference" "#PWR041" (id 0) (at 207.518 120.65 0)
+      (effects (font (size 1.27 1.27)) hide)
+    )
+    (property "Value" "VCC" (id 1) (at 201.93 115.824 0)
+      (effects (font (size 1.27 1.27)) (justify left))
+    )
+    (property "Footprint" "" (id 2) (at 207.518 116.84 0)
+      (effects (font (size 1.27 1.27)) hide)
+    )
+    (property "Datasheet" "" (id 3) (at 207.518 116.84 0)
+      (effects (font (size 1.27 1.27)) hide)
+    )
+    (pin "1")
+  )
   (symbol (lib_id "power:VCC") (at 146.304 197.358 0) (unit 1)
     (in_bom yes) (on_board yes)
@@
     (pin "1")
   )
+  (symbol (lib_id "power:VCC") (at 174.752 116.84 0) (unit 1)
+    (in_bom yes) (on_board yes)
+    (property "Reference" "#PWR040" (id 0) (at 174.752 120.65 0)
+      (effects (font (size 1.27 1.27)) hide)
+    )
+    (property "Value" "VCC" (id 1) (at 169.164 115.824 0)
+      (effects (font (size 1.27 1.27)) (justify left))
+    )
+    (property "Footprint" "" (id 2) (at 174.752 116.84 0)
+      (effects (font (size 1.27 1.27)) hide)
+    )
+    (property "Datasheet" "" (id 3) (at 174.752 116.84 0)
+      (effects (font (size 1.27 1.27)) hide)
+    )
+    (pin "1")
+  )
   (symbol (lib_id "power:GND") (at 44.704 136.398 270) (unit 1)
     (in_bom yes) (on_board yes) (fields_autoplaced)
@@
     (pin "6")
   )
-  (symbol (lib_id "Connector:TestPoint") (at 174.752 116.84 0) (mirror y) (unit 1)
-    (in_bom yes) (on_board yes)
-    (property "Reference" "TP5" (id 0) (at 168.91 113.284 0)
-      (effects (font (size 1.27 1.27)) (justify right))
-    )
-    (property "Value" "TestPoint" (id 1) (at 165.1 115.316 0)
-      (effects (font (size 1.27 1.27)) (justify right))
-    )
-    (property "Footprint" "TestPoint:TestPoint_THTPad_1.0x1.0mm_Drill0.5mm" (id 2) (at 169.672 116.84 0)
-      (effects (font (size 1.27 1.27)) hide)
-    )
-    (property "Datasheet" "~" (id 3) (at 169.672 116.84 0)
-      (effects (font (size 1.27 1.27)) hide)
-    )
-    (pin "1")
-  )
   (symbol (lib_id "Device:R") (at 142.494 199.898 90) (unit 1)
