File: Color Magic/pwr_S100buss.kicad_sch (KiCad schematic)
At the start: 39 parts, among them P1 S100_MALE, U14 LM7805K, U49 LM7812

Commit message: Add files via upload
Connections:
- net GND: no longer H1.1 (Pin_1), H2.1 (Pin_1)
- no-connect marks 33 -> 35
Other:
- moved on the sheet: C35, C36, U49

Commit message: Add files via upload
Updated to current version. Still plotting...
Parts:
- removed U49: LM7812, Package_TO_SOT_THT:TO-92, symbol Regulator_Linear:LM7812_TO220
- added U49: LM78L12, Package_TO_SOT_THT:TO-92L, symbol Regulator_Linear:LM78L12_TO92
Connections:
- net +12V: now also U49.1 (VO)
- net BUS16V: now also U49.3 (VI)
- net GND: now also U49.2 (GND)
Changed lines of the file:
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@@
   (title_block
     (title "Lomas Color Magic Redux")
-    (date "2023-04-14")
-    (rev "1.0-001")
+    (date "2024-02-15")
+    (rev "1.1-001")
     (company "Lomas Data Produtcs")
     (comment 1 "Redraw/modifications (c) Richard A. Cini")
@@
   )
   (junction (at 243.84 153.67) (diameter 0) (color 0 0 0 0)
-  )
-  (junction (at 61.722 102.87) (diameter 0) (color 0 0 0 0)
   )
   (junction (at 163.83 138.43) (diameter 0) (color 0 0 0 0)
@@
     (stroke (width 0) (type default) (color 0 0 0 0))
   )
-  (wire (pts (xy 61.722 102.87) (xy 68.834 102.87))
-    (stroke (width 0) (type default) (color 0 0 0 0))
-  )
   (wire (pts (xy 119.126 59.69) (xy 119.126 44.45))
     (stroke (width 0) (type default) (color 0 0 0 0))
@@
   )
   (wire (pts (xy 232.41 130.81) (xy 243.84 130.81))
-    (stroke (width 0) (type default) (color 0 0 0 0))
-  )
-  (wire (pts (xy 52.832 113.03) (xy 69.088 113.03))
     (stroke (width 0) (type default) (color 0 0 0 0))
   )
@@
     (effects (font (size 1.524 1.524)) (justify left bottom))
   )
-  (label "ZERO" (at 62.738 113.03 0)
-    (effects (font (size 1.27 1.27)) (justify left bottom))
-  )
   (label "PWRFAIL*" (at 55.626 58.42 90)
     (effects (font (size 1.524 1.524)) (justify left bottom))
-  )
-  (label "ONE" (at 64.262 102.87 0)
-    (effects (font (size 1.27 1.27)) (justify left bottom))
   )
   (label "sHLTA" (at 144.526 58.42 90)
@@
     (pin "2")
   )
-  (symbol (lib_id "Regulator_Linear:LM7812_TO220") (at 118.618 102.87 0) (unit 1)
-    (in_bom yes) (on_board yes) (fields_autoplaced)
-    (property "Reference" "U49" (id 0) (at 118.618 97.2652 0))
-    (property "Value" "LM7812" (id 1) (at 118.618 99.8021 0))
-    (property "Footprint" "Package_TO_SOT_THT:TO-92" (id 2) (at 118.618 97.155 0)
-      (effects (font (size 1.27 1.27) italic) hide)
-    )
-    (property "Datasheet" "https://www.onsemi.cn/PowerSolutions/document/MC7800-D.PDF" (id 3) (at 118.618 104.14 0)
-      (effects (font (size 1.27 1.27)) hide)
-    )
-    (pin "1")
-    (pin "2")
-    (pin "3")
-  )
   (symbol (lib_id "power:VCC") (at 61.722 102.87 0) (unit 1)
     (in_bom yes) (on_board yes) (fields_autoplaced)
@@
     (pin "1")
   )
+  (symbol (lib_id "Regulator_Linear:LM78L12_TO92") (at 118.618 102.87 0) (unit 1)
+    (in_bom yes) (on_board yes) (fields_autoplaced)
+    (property "Reference" "U49" (id 0) (at 118.618 97.2652 0))
+    (property "Value" "LM78L12" (id 1) (at 118.618 99.8021 0))
+    (property "Footprint" "Package_TO_SOT_THT:TO-92L" (id 2) (at 118.618 97.155 0)
+      (effects (font (size 1.27 1.27) italic) hide)
+    )
+    (property "Datasheet" "https://www.onsemi.com/pub/Collateral/MC78L06A-D.pdf" (id 3) (at 118.618 104.14 0)
+      (effects (font (size 1.27 1.27)) hide)
+    )
+    (pin "1")
+    (pin "2")
+    (pin "3")
+  )
   (symbol (lib_id "Device:C") (at 186.69 165.1 0) (unit 1)

Commit message: Add files via upload
Connections:
- no-connect marks 35 -> 34
Changed lines of the file:
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@@
   (title_block
     (title "Lomas Color Magic Redux")
-    (date "2024-02-15")
-    (rev "1.1-001")
+    (date "2024-06-08")
+    (rev "1.1-003")
     (company "Lomas Data Produtcs")
     (comment 1 "Redraw/modifications (c) Richard A. Cini")
@@
   (no_connect (at 164.846 59.69))
   (no_connect (at 197.866 59.69))
-  (no_connect (at 274.066 59.69))
   (no_connect (at 70.866 59.69))
   (no_connect (at 271.526 59.69))
@@
     (effects (font (size 1.524 1.524)) (justify left bottom))
   )
-  (label "POC*" (at 274.066 58.42 90)
-    (effects (font (size 1.524 1.524)) (justify left bottom))
-  )
   (label "INT*" (at 208.026 58.42 90)
     (effects (font (size 1.524 1.524)) (justify left bottom))
@@
       (effects (font (size 1.27 1.27)) (justify right) hide)
     )
+  )
+  (global_label "POC*" (shape output) (at 274.066 59.69 270) (fields_autoplaced)
+    (effects (font (size 1.27 1.27)) (justify right))
+    (property "Intersheet References" "${INTERSHEET_REFS}" (id 0) (at 273.9866 66.8523 90)
+      (effects (font (size 1.27 1.27)) (justify right) hide)
+    )

Commit message: Add files via upload
Parts:
- P1: symbol RAC_Custom2:S100_MALE -> RAC_Custom:S100_MALE
- U14: symbol RAC_Custom2:LM7805K -> RAC_Custom:LM7805K
Connections:
- net 0V_A is gone; now on net GND: P1.20 (0_V1)
- net 0V_B is gone; now on net GND: P1.53 (0_V3)
- net 0V_C is gone; now on net GND: P1.70 (0_V4)
- no-connect marks 34 -> 31
Other:
- note added: "NOTE: Original board used adjustible regulators rather than fixed. So R19 (1.3k) and R20 (160) on the LM317(7812) are not used, and R12 (470) and R13 (150) on the LM338 (7805K) are not used."
- note added: "NOTE: Pins 20, 53, and 70 are grounded to be compliant with IEEE-696 (post-Altair/IMSAI or any front-panel based system)."
- note removed: "NOTE: Original board used adjustible regulators rather than fixed. So R19 (1.3k) and R20 (160) on the LM317(7812) is not used and R12 (470) and R13 (150) on the LM338 (7805K) is not used."
- moved on the sheet: C1, C10, C11, C12, C13, C14, C15, C16, C17, C18, C20, C21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
