File: Color Magic/timing.kicad_sch (KiCad schematic)
At the start: 31 parts, among them J1 CGA VIdeo Out, J2 RCJ-014, Q1 2N3904, U1 PAL16L8, U10 74LS365, U11 74LS244, U12 74LS151, U13 74LS74, U19 74LS04, U20 74LS175, U21 74LS86, U22 74LS02, U30 74LS04, U31 74LS32, U32 74LS04, U33 74LS00, U34 74ALS174, U35 74LS164, U36 74LS74, U5 74LS273, U6 74LS393, U9 74LS08

Commit message: Add files via upload
Connections:
- net GND: no longer U10.1 (E1), U10.15 (E2), U11.1 (OEa), U11.19 (OEb), U6.12 (MR), U6.2 (MR)
- net VCC: no longer U12.12 (I7), U20.4 (D0), U34.1 (~{Mr}), U35.1 (A), U35.2 (B), U5.1 (~{Mr})
- new net ONE: U12.12 (I7), U20.4 (D0), U34.1 (~{Mr}), U35.1 (A), U35.2 (B), U5.1 (~{Mr})
- new net ZERO: U10.1 (E1), U10.15 (E2), U11.1 (OEa), U11.19 (OEb), U6.12 (MR), U6.2 (MR)
Changed lines of the file:
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@@
   (title_block
     (title "Lomas Color Magic Redux")
-    (date "2023-03-04")
+    (date "2023-04-14")
     (rev "1.0-001")
     (company "Lomas Data Produtcs")
@@
   (junction (at 84.836 233.426) (diameter 0) (color 0 0 0 0)
   )
-  (junction (at 271.78 118.872) (diameter 0) (color 0 0 0 0)
-  )
   (junction (at 310.642 108.204) (diameter 0) (color 0 0 0 0)
   )
@@
   (junction (at 67.056 194.31) (diameter 0) (color 0 0 0 0)
   )
-  (junction (at 37.846 215.138) (diameter 0) (color 0 0 0 0)
-  )
   (junction (at 103.378 233.426) (diameter 0) (color 0 0 0 0)
   )
@@
   (junction (at 26.924 258.826) (diameter 0) (color 0 0 0 0)
   )
-  (junction (at 233.426 59.69) (diameter 0) (color 0 0 0 0)
-  )
   (junction (at 213.614 39.37) (diameter 0) (color 0 0 0 0)
   )
@@
   (junction (at 299.466 90.932) (diameter 0) (color 0 0 0 0)
   )
-  (junction (at 246.126 67.31) (diameter 0) (color 0 0 0 0)
-  )
   (junction (at 237.998 179.07) (diameter 0) (color 0 0 0 0)
-  )
-  (junction (at 39.116 94.996) (diameter 0) (color 0 0 0 0)
-  )
-  (junction (at 259.08 111.252) (diameter 0) (color 0 0 0 0)
   )
   (junction (at 211.582 179.07) (diameter 0) (color 0 0 0 0)
@@
     (stroke (width 0) (type default) (color 0 0 0 0))
   )
-  (wire (pts (xy 271.78 118.872) (xy 259.08 118.872))
-    (stroke (width 0) (type default) (color 0 0 0 0))
-  )
   (wire (pts (xy 46.99 233.426) (xy 46.99 235.966))
     (stroke (width 0) (type default) (color 0 0 0 0))
@@
     (stroke (width 0) (type default) (color 0 0 0 0))
   )
-  (wire (pts (xy 259.08 118.872) (xy 259.08 111.252))
-    (stroke (width 0) (type default) (color 0 0 0 0))
-  )
   (wire (pts (xy 294.894 189.738) (xy 294.894 202.184))
     (stroke (width 0) (type default) (color 0 0 0 0))
@@
     (stroke (width 0) (type default) (color 0 0 0 0))
   )
-  (wire (pts (xy 246.126 67.31) (xy 233.426 67.31))
-    (stroke (width 0) (type default) (color 0 0 0 0))
-  )
   (wire (pts (xy 41.656 194.31) (xy 37.846 194.31))
     (stroke (width 0) (type default) (color 0 0 0 0))
@@
   )
   (wire (pts (xy 67.056 107.696) (xy 74.676 107.696))
-    (stroke (width 0) (type default) (color 0 0 0 0))
-  )
-  (wire (pts (xy 233.426 67.31) (xy 233.426 59.69))
     (stroke (width 0) (type default) (color 0 0 0 0))
   )
@@
     (effects (font (size 1.27 1.27)) (justify left bottom))
   )
+  (label "ZERO" (at 37.846 194.31 180)
+    (effects (font (size 1.27 1.27)) (justify right bottom))
+  )
+  (label "ONE" (at 39.116 92.456 180)
+    (effects (font (size 1.27 1.27)) (justify right bottom))
+  )
+  (label "ONE" (at 39.624 131.572 180)
+    (effects (font (size 1.27 1.27)) (justify right bottom))
+  )
+  (label "ONE" (at 176.276 59.69 180)
+    (effects (font (size 1.27 1.27)) (justify right bottom))
+  )
+  (label "ONE" (at 310.896 192.278 180)
+    (effects (font (size 1.27 1.27)) (justify right bottom))
+  )
+  (label "ZERO" (at 259.08 108.712 180)
+    (effects (font (size 1.27 1.27)) (justify right bottom))
+  )
+  (label "ZERO" (at 233.426 57.15 180)
+    (effects (font (size 1.27 1.27)) (justify right bottom))
+  )
+  (label "ONE" (at 52.832 59.182 180)
+    (effects (font (size 1.27 1.27)) (justify right bottom))
+  )
   (global_label "{slash}3.6MCLK" (shape input) (at 52.832 54.102 180) (fields_autoplaced)
     (effects (font (size 1.27 1.27)) (justify right))
@@
     (pin "14")
     (pin "7")
-  )
-  (symbol (lib_id "power:VCC") (at 39.116 94.996 90) (unit 1)
-    (in_bom yes) (on_board yes)
-    (property "Reference" "#PWR0604" (id 0) (at 42.926 94.996 0)
-      (effects (font (size 1.27 1.27)) hide)
-    )
-    (property "Value" "VCC" (id 1) (at 32.258 94.996 90)
-      (effects (font (size 1.27 1.27)) (justify right))
-    )
-    (property "Footprint" "" (id 2) (at 39.116 94.996 0)
-      (effects (font (size 1.27 1.27)) hide)
-    )
-    (property "Datasheet" "" (id 3) (at 39.116 94.996 0)
-      (effects (font (size 1.27 1.27)) hide)
-    )
-    (pin "1")
   )
   (symbol (lib_id "Device:R") (at 288.29 96.012 90) (unit 1)
@@
     (pin "9")
   )
-  (symbol (lib_id "power:VCC") (at 52.832 59.182 90) (unit 1)
-    (in_bom yes) (on_board yes)
-    (property "Reference" "#PWR0608" (id 0) (at 56.642 59.182 0)
-      (effects (font (size 1.27 1.27)) hide)
-    )
-    (property "Value" "VCC" (id 1) (at 46.482 59.182 90)
-      (effects (font (size 1.27 1.27)) (justify right))
-    )
-    (property "Footprint" "" (id 2) (at 52.832 59.182 0)
-      (effects (font (size 1.27 1.27)) hide)
-    )
-    (property "Datasheet" "" (id 3) (at 52.832 59.182 0)
-      (effects (font (size 1.27 1.27)) hide)
-    )
-    (pin "1")
-  )
   (symbol (lib_id "74xx:74LS74") (at 122.174 246.126 0) (unit 3)
     (in_bom yes) (on_board yes) (fields_autoplaced)
@@
     (pin "7")
   )
-  (symbol (lib_id "power:VCC") (at 176.276 59.69 90) (unit 1)
-    (in_bom yes) (on_board yes)
-    (property "Reference" "#PWR0613" (id 0) (at 180.086 59.69 0)
-      (effects (font (size 1.27 1.27)) hide)
-    )
-    (property "Value" "VCC" (id 1) (at 169.418 59.944 90)
-      (effects (font (size 1.27 1.27)) (justify right))
-    )
-    (property "Footprint" "" (id 2) (at 176.276 59.69 0)
-      (effects (font (size 1.27 1.27)) hide)
-    )
-    (property "Datasheet" "" (id 3) (at 176.276 59.69 0)
-      (effects (font (size 1.27 1.27)) hide)
-    )
-    (pin "1")
-  )
   (symbol (lib_id "power:GND") (at 188.976 67.31 0) (unit 1)
     (in_bom yes) (on_board yes) (fields_autoplaced)
@@
     )
     (property "Datasheet" "" (id 3) (at 188.976 67.31 0)
-      (effects (font (size 1.27 1.27)) hide)
-    )
-    (pin "1")
-  )
-  (symbol (lib_id "power:VCC") (at 310.896 192.278 90) (unit 1)
-    (in_bom yes) (on_board yes)
-    (property "Reference" "#PWR0624" (id 0) (at 314.706 192.278 0)
-      (effects (font (size 1.27 1.27)) hide)
-    )
-    (property "Value" "VCC" (id 1) (at 303.784 192.532 90)
-      (effects (font (size 1.27 1.27)) (justify right))
-    )
-    (property "Footprint" "" (id 2) (at 310.896 192.278 0)
-      (effects (font (size 1.27 1.27)) hide)
-    )
-    (property "Datasheet" "" (id 3) (at 310.896 192.278 0)
       (effects (font (size 1.27 1.27)) hide)
     )
@@
     (pin "1")
   )
-  (symbol (lib_id "power:GND") (at 37.846 215.138 0) (unit 1)
-    (in_bom yes) (on_board yes) (fields_autoplaced)
-    (property "Reference" "#PWR0603" (id 0) (at 37.846 221.488 0)
-      (effects (font (size 1.27 1.27)) hide)
-    )
-    (property "Value" "GND" (id 1) (at 37.846 219.5814 0))
-    (property "Footprint" "" (id 2) (at 37.846 215.138 0)
-      (effects (font (size 1.27 1.27)) hide)
-    )
-    (property "Datasheet" "" (id 3) (at 37.846 215.138 0)
-      (effects (font (size 1.27 1.27)) hide)
-    )
-    (pin "1")
-  )
   (symbol (lib_id "74xx:74LS74") (at 271.526 189.23 0) (unit 1)
     (in_bom yes) (on_board yes) (fields_autoplaced)
@@
     (pin "2")
   )
-  (symbol (lib_id "power:VCC") (at 39.624 131.572 90) (unit 1)
-    (in_bom yes) (on_board yes)
-    (property "Reference" "#PWR0605" (id 0) (at 43.434 131.572 0)
-      (effects (font (size 1.27 1.27)) hide)
-    )
-    (property "Value" "VCC" (id 1) (at 32.766 131.572 90)
-      (effects (font (size 1.27 1.27)) (justify right))
-    )
-    (property "Footprint" "" (id 2) (at 39.624 131.572 0)
-      (effects (font (size 1.27 1.27)) hide)
-    )
-    (property "Datasheet" "" (id 3) (at 39.624 131.572 0)
-      (effects (font (size 1.27 1.27)) hide)
-    )
-    (pin "1")
-  )
   (symbol (lib_id "74xx:74LS393") (at 54.356 189.23 0) (unit 2)

Commit message: Add files via upload
Updated to current version. Still plotting...
Parts:
- removed U35: 74LS164, Package_DIP:DIP-14_W7.62mm_Socket_LongPads, symbol 74xx_IEEE:74164
- added U35: 74LS164, Package_DIP:DIP-14_W7.62mm_Socket, symbol 74xx:74HC164
- R10, R11, R9: footprint Resistor_THT:R_Axial_DIN0204_L3.6mm_D1.6mm_P5.08mm_Horizontal -> Resistor_THT:R_Axial_DIN0207_L6.3mm_D2.5mm_P7.62mm_Horizontal
- U1, U11, U5: footprint Package_DIP:DIP-20_W7.62mm_Socket_LongPads -> Package_DIP:DIP-20_W7.62mm_Socket
- U10, U12, U20, U34: footprint Package_DIP:DIP-16_W7.62mm_Socket_LongPads -> Package_DIP:DIP-16_W7.62mm_Socket
- U13, U19, U21, U22, U30, U31, U32, U33, U36, U6, U9: footprint Package_DIP:DIP-14_W7.62mm_Socket_LongPads -> Package_DIP:DIP-14_W7.62mm_Socket
Connections:
- net ONE is gone; now on net VCC: U12.12 (I7), U20.4 (D0), U34.1 (~{Mr}), U5.1 (~{Mr})
- net ZERO is gone; now on net GND: U10.1 (E1), U10.15 (E2), U11.1 (OEa), U11.19 (OEb), U6.12 (MR), U6.2 (MR)
- net GND: now also U35.7 (GND)
- net LCLK: now also U35.8 (CP)
- net U35.12: now also U35.12 (Q6)
- net U35.13: now also U35.13 (Q7)
- net VCC: now also U35.1 (DSA), U35.14 (VCC), U35.2 (DSB)
- net /HSYNC_DLY: now also U35.9 (~{MR})
- net at U21.10: now also U35.4 (Q1)
- net at U21.9: now also U35.11 (Q5)
Other:
- note added: "NOTE: schematic typo on pin 4 (called pin 10)."
- note removed: "NOTE: Need to check pins 1 and 4. Typo in schematic?"
- moved on the sheet: U19D, U21B, U21C

Commit message: Add files via upload
Parts:
- J1: value CGA VIdeo Out -> CGA Out
Other:
- note added: "BLUE"
- note added: "CYAN"
- note added: "GREEN"
- note added: "MAGENTA"
- note added: "RED"
- note added: "YELLOW_BURST"
- note removed: "NOTE: Need to check device number."
- note removed: "NOTE: schematic typo on pin 4 (called pin 10)."
Changed lines of the file:
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@@
   (title_block
     (title "Lomas Color Magic Redux")
-    (date "2024-02-15")
-    (rev "1.1-001")
+    (date "2024-06-08")
+    (rev "1.1-003")
     (company "Lomas Data Produtcs")
     (comment 1 "Redraw/modifications (c) Richard A. Cini")
@@
   (junction (at 299.466 98.552) (diameter 0) (color 0 0 0 0)
   )
-  (junction (at 323.596 215.138) (diameter 0) (color 0 0 0 0)
-  )
   (junction (at 266.446 52.07) (diameter 0) (color 0 0 0 0)
   )
   (junction (at 95.504 36.322) (diameter 0) (color 0 0 0 0)
   )
-  (junction (at 310.896 207.518) (diameter 0) (color 0 0 0 0)
-  )
   (junction (at 26.924 233.426) (diameter 0) (color 0 0 0 0)
   )
@@
   )
   (junction (at 299.466 96.012) (diameter 0) (color 0 0 0 0)
+  )
+  (junction (at 301.244 207.518) (diameter 0) (color 0 0 0 0)
   )
   (junction (at 67.056 194.31) (diameter 0) (color 0 0 0 0)
@@
     (stroke (width 0) (type default) (color 0 0 0 0))
   )
-  (wire (pts (xy 304.8 187.198) (xy 310.896 187.198))
-    (stroke (width 0) (type default) (color 0 0 0 0))
-  )
   (wire (pts (xy 31.242 136.652) (xy 31.242 118.11))
     (stroke (width 0) (type default) (color 0 0 0 0))
@@
     (stroke (width 0) (type default) (color 0 0 0 0))
   )
-  (wire (pts (xy 279.146 186.69) (xy 304.8 186.69))
-    (stroke (width 0) (type default) (color 0 0 0 0))
-  )
   (wire (pts (xy 78.232 38.862) (xy 94.488 38.862))
     (stroke (width 0) (type default) (color 0 0 0 0))
@@
     (stroke (width 0) (type default) (color 0 0 0 0))
   )
+  (wire (pts (xy 288.036 186.69) (xy 279.146 186.69))
+    (stroke (width 0) (type default) (color 0 0 0 0))
+  )
   (wire (pts (xy 203.962 179.07) (xy 211.582 179.07))
     (stroke (width 0) (type default) (color 0 0 0 0))
@@
     (stroke (width 0) (type default) (color 0 0 0 0))
   )
+  (wire (pts (xy 288.036 187.198) (xy 288.036 186.69))
+    (stroke (width 0) (type default) (color 0 0 0 0))
+  )
   (wire (pts (xy 92.202 100.584) (xy 92.202 134.112))
     (stroke (width 0) (type default) (color 0 0 0 0))
   )
+  (wire (pts (xy 310.896 187.198) (xy 288.036 187.198))
+    (stroke (width 0) (type default) (color 0 0 0 0))
+  )
   (wire (pts (xy 41.656 41.656) (xy 41.656 38.862))
     (stroke (width 0) (type default) (color 0 0 0 0))
@@
     (stroke (width 0) (type default) (color 0 0 0 0))
   )
+  (wire (pts (xy 301.244 207.518) (xy 301.244 211.582))
+    (stroke (width 0) (type default) (color 0 0 0 0))
+  )
   (wire (pts (xy 299.466 101.092) (xy 299.466 98.552))
     (stroke (width 0) (type default) (color 0 0 0 0))
   )
-  (wire (pts (xy 310.896 215.138) (xy 310.896 207.518))
-    (stroke (width 0) (type default) (color 0 0 0 0))
-  )
   (wire (pts (xy 213.614 27.432) (xy 213.614 39.37))
     (stroke (width 0) (type default) (color 0 0 0 0))
@@
     (stroke (width 0) (type default) (color 0 0 0 0))
   )
-  (wire (pts (xy 304.8 186.69) (xy 304.8 187.198))
-    (stroke (width 0) (type default) (color 0 0 0 0))
-  )
-  (wire (pts (xy 323.596 215.138) (xy 310.896 215.138))
-    (stroke (width 0) (type default) (color 0 0 0 0))
-  )
   (wire (pts (xy 237.998 179.07) (xy 271.526 179.07))
     (stroke (width 0) (type default) (color 0 0 0 0))
@@
     (stroke (width 0) (type default) (color 0 0 0 0))
   )
-  (text "NOTE: schematic typo on pin 4 (called pin 10)." (at 136.398 165.608 0)
+  (text "CYAN" (at 302.768 182.118 0)
+    (effects (font (size 1.27 1.27)) (justify left bottom))
+  )
+  (text "RED" (at 303.022 184.658 0)
+    (effects (font (size 1.27 1.27)) (justify left bottom))
+  )
+  (text "YELLOW_BURST" (at 295.91 189.738 0)
     (effects (font (size 1.27 1.27)) (justify left bottom))
   )
@@
     (effects (font (size 1.27 1.27)) (justify left bottom))
   )
-  (text "NOTE: Need to check device number." (at 185.674 176.022 0)
+  (text "BLUE" (at 303.022 176.784 0)
+    (effects (font (size 1.27 1.27)) (justify left bottom))
+  )
+  (text "MAGENTA" (at 301.752 187.198 0)
+    (effects (font (size 1.27 1.27)) (justify left bottom))
+  )
+  (text "GREEN" (at 302.768 179.578 0)
     (effects (font (size 1.27 1.27)) (justify left bottom))
   )
@@
     (pin "7")
   )
+  (symbol (lib_id "power:GND") (at 301.244 211.582 0) (unit 1)
+    (in_bom yes) (on_board yes) (fields_autoplaced)
+    (property "Reference" "#PWR034" (id 0) (at 301.244 217.932 0)
+      (effects (font (size 1.27 1.27)) hide)
+    )
+    (property "Value" "GND" (id 1) (at 301.244 216.0254 0))
+    (property "Footprint" "" (id 2) (at 301.244 211.582 0)
+      (effects (font (size 1.27 1.27)) hide)
+    )
+    (property "Datasheet" "" (id 3) (at 301.244 211.582 0)
+      (effects (font (size 1.27 1.27)) hide)
+    )
+    (pin "1")
+  )
   (symbol (lib_id "power:GND") (at 188.976 67.31 0) (unit 1)
     (in_bom yes) (on_board yes) (fields_autoplaced)
@@
     (in_bom yes) (on_board yes) (fields_autoplaced)
     (property "Reference" "J1" (id 0) (at 299.466 29.5742 0))
-    (property "Value" "CGA VIdeo Out" (id 1) (at 299.466 32.1111 0))
+    (property "Value" "CGA Out" (id 1) (at 299.466 32.1111 0))
     (property "Footprint" "Connector_PinHeader_2.54mm:PinHeader_2x05_P2.54mm_Vertical" (id 2) (at 298.196 39.624 0)
       (effects (font (size 1.27 1.27)) hide)

Commit message: Add files via upload
Parts:
- added TP2: TestPoint, TestPoint:TestPoint_THTPad_1.0x1.0mm_Drill0.5mm, symbol Connector:TestPoint
- U10: value 74LS365 -> 74LS367
Connections:
- net /BW: no longer U36.4 (~{S})
- net U12.5 renamed COLOR_COMPOSITE
- net U19.8 renamed COMPOSITE_SYNC
- new net: TP2.1, U36.4 (~{S})
Other:
- note added: "NOTE: Pin 4 should connect to /BW but it connects nowhere on the prototype. It would be odd for /S to be left floating, though."
- note added: "NOTE: R2/3/4 unpopulated. B&W Composite"
- note removed: "NOTE: R2/3/4 unpopulated."
- moved on the sheet: J1, J2, Q1, R1, R10, R11, R2, R3, R4, R5, R6, R9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

Commit message: Add files via upload
Other:
- note added: "TP2: Pin 4 is misdrawn on the LDP schematics - it is shown as pin 10 and connects to /BW. The IBM CGA card also has it connected to /BW. TIE TO /BW."
- note removed: "NOTE: Pin 4 should connect to /BW but it connects nowhere on the prototype. It would be odd for /S to be left floating, though."
Changed lines of the file:
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@@
     (effects (font (size 1.27 1.27)) (justify left bottom))
   )
-  (text "NOTE: Pin 4 should connect to /BW but it\nconnects nowhere on the prototype. It would\nbe odd for /S to be left floating, though."
-    (at 138.43 168.148 0)
+  (text "TP2: Pin 4 is misdrawn on the LDP schematics - \nit is shown as pin 10 and connects to /BW. The\nIBM CGA card also has it connected to /BW.\nTIE TO /BW.\n"
+    (at 141.478 172.974 0)
     (effects (font (size 1.27 1.27)) (justify left bottom))
   )

Commit message: Add files via upload
Final versions uploaded.
Parts:
- removed TP2: TestPoint, TestPoint:TestPoint_THTPad_1.0x1.0mm_Drill0.5mm, symbol Connector:TestPoint
Connections:
- net /BW: now also U36.4 (~{S})
Changed lines of the file:
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@@
   (title_block
     (title "Lomas Color Magic Redux")
-    (date "2024-08-16")
-    (rev "1.1-004")
+    (date "2024-09-24")
+    (rev "1.1-005")
     (company "Lomas Data Produtcs")
     (comment 1 "Redraw/modifications (c) Richard A. Cini")
@@
     (stroke (width 0) (type default) (color 0 0 0 0))
   )
+  (wire (pts (xy 164.592 140.462) (xy 164.592 138.176))
+    (stroke (width 0) (type default) (color 0 0 0 0))
+  )
   (wire (pts (xy 122.174 256.286) (xy 122.174 258.826))
     (stroke (width 0) (type default) (color 0 0 0 0))
@@
   )
   (wire (pts (xy 359.918 93.218) (xy 359.918 90.678))
+    (stroke (width 0) (type default) (color 0 0 0 0))
+  )
+  (wire (pts (xy 164.592 138.176) (xy 156.718 138.176))
     (stroke (width 0) (type default) (color 0 0 0 0))
   )
@@
     (property "Intersheet References" "${INTERSHEET_REFS}" (id 0) (at 142.7257 97.9646 0)
       (effects (font (size 1.27 1.27)) (justify left) hide)
+    )
+  )
+  (global_label "{slash}BW" (shape input) (at 156.718 138.176 180) (fields_autoplaced)
+    (effects (font (size 1.27 1.27)) (justify right))
+    (property "Intersheet References" "${INTERSHEET_REFS}" (id 0) (at 150.3419 138.0966 0)
+      (effects (font (size 1.27 1.27)) (justify right) hide)
     )
   )
@@
       (effects (font (size 1.27 1.27)) hide)
     )
-    (pin "1")
-  )
-  (symbol (lib_id "Connector:TestPoint") (at 164.592 140.462 0) (mirror y) (unit 1)
-    (in_bom yes) (on_board yes)
-    (property "Reference" "TP2" (id 0) (at 158.75 136.906 0)
-      (effects (font (size 1.27 1.27)) (justify right))
-    )
-    (property "Value" "TestPoint" (id 1) (at 154.94 138.938 0)
-      (effects (font (size 1.27 1.27)) (justify right))
-    )
-    (property "Footprint" "TestPoint:TestPoint_THTPad_1.0x1.0mm_Drill0.5mm" (id 2) (at 159.512 140.462 0)
-      (effects (font (size 1.27 1.27)) hide)
-    )
-    (property "Datasheet" "~" (id 3) (at 159.512 140.462 0)
-      (effects (font (size 1.27 1.27)) hide)
-    )
