File: Color Magic/vidgen.kicad_sch (KiCad schematic)
At the start: 27 parts, among them U15 74LS153, U17 74LS174, U19 74LS04, U2 74LS273, U23 2764, U24 74LS273, U26 MC6845, U27 74LS166, U3 74LS153, U32 74LS04, U38 74LS174, U4 74LS166, U44 74LS244, U45 74LS244, U47 74LS244, U48 74LS244, U50 74LS166, U9 74LS08

Commit message: Add files via upload
Connections:
- net GND: no longer JP1.2 (Pin_2), JP1.4 (Pin_4), JP1.6 (Pin_6), JP1.8 (Pin_8), JP2.2 (B), JP4.2 (B), U23.20 (~{CE}), U23.22 (~{OE}), U27.1 (Ds), U27.6 (CE), U4.1 (Ds), U4.6 (CE), U50.1 (Ds), U50.6 (CE)
- net VCC: no longer JP401.2 (B), R15.1, R17.1, RN1.1 (common), U24.1 (~{Mr})
- new net ONE: JP401.2 (B), R15.1, R17.1, RN1.1 (common), U24.1 (~{Mr})
- new net ZERO: JP1.2 (Pin_2), JP1.4 (Pin_4), JP1.6 (Pin_6), JP1.8 (Pin_8), JP2.2 (B), JP4.2 (B), U23.20 (~{CE}), U23.22 (~{OE}), U27.1 (Ds), U27.6 (CE), U4.1 (Ds), U4.6 (CE), U50.1 (Ds), U50.6 (CE)

Commit message: Add files via upload
Updated to current version. Still plotting...
Parts:
- R15, R17: footprint Resistor_THT:R_Axial_DIN0204_L3.6mm_D1.6mm_P5.08mm_Horizontal -> Resistor_THT:R_Axial_DIN0207_L6.3mm_D2.5mm_P7.62mm_Horizontal
- U15, U17, U27, U3, U38, U4, U50: footprint Package_DIP:DIP-16_W7.62mm_Socket_LongPads -> Package_DIP:DIP-16_W7.62mm_Socket
- U19, U32, U9: footprint Package_DIP:DIP-14_W7.62mm_Socket_LongPads -> Package_DIP:DIP-14_W7.62mm_Socket
- U2, U24, U44, U45, U47, U48: footprint Package_DIP:DIP-20_W7.62mm_Socket_LongPads -> Package_DIP:DIP-20_W7.62mm_Socket
Connections:
- net ONE is gone; now on net VCC: JP401.2 (B), R15.1, R17.1, RN1.1 (common), U24.1 (~{Mr})
- net ZERO is gone; now on net GND: JP1.2 (Pin_2), JP1.4 (Pin_4), JP1.6 (Pin_6), JP1.8 (Pin_8), JP2.2 (B), JP4.2 (B), U23.20 (~{CE}), U23.22 (~{OE}), U27.1 (Ds), U27.6 (CE), U4.1 (Ds), U4.6 (CE), U50.1 (Ds), U50.6 (CE)
- net CGRDM11 renamed CGROM11
- net CGRDM12 renamed CGROM12
Other:
- note added: "NOTE: Check pin 1 connection. "+5VS" not noted anywhere."
- note removed: "NOTE: Check pin 1 connection."
- moved on the sheet: U32F

Commit message: Add files via upload
Connections:
- net 2C1: no longer names the net of U15.11 (I1b), U9.3
- net BW: no longer names the net of U17.7 (Q2), U32.13
Other:
- note added: "2764A: JP2 - Closed JP3 - Open JP4 - Closed JP5 - Open"
- note added: "BW"
- note added: "Default for 2732: JP2 - Open JP3 - Open JP4 - Closed JP5 - Open"
- note added: "NOTE: The Color Magic uses an Intel D2732A (200nS). The board seems particularly sensitive to what brand/type of 2732 is used (I tried AMD, Fujitsu, and Hitachi with no success). I switched to an AMD2764A and it worked fine."
- note added: "NOTE: hanging line on U9.1"
- note removed: "Default: JP2 - Open JP3 - Open JP4 - Closed JP5 - Open"
- note removed: "NOTE: Check pin 1 connection. "+5VS" not noted anywhere."
- note removed: "NOTE: Need to check A0-A2 connection to 6845 as A0 and A2 are drawn reversed."
- note removed: "NOTE: pin 10 could be AT2. Check."
- moved on the sheet: U15, U3, U32F, U4, U50, U9A

Commit message: Add files via upload
Connections:
- net AT7: now also U9.2; no longer U9.1
- net /ENABLE_BLINK: now also U9.1; no longer U9.2
- net BW: now reaches U17.7 (Q2), U32.13
- net PU_RN1_8: now reaches RN1.8 (R7)
- net MDO0 renamed MD0
- net MDO1 renamed MD1
- net MDO10 renamed MD10
- net MDO11 renamed MD11
- net MDO12 renamed MD12
- net MDO13 renamed MD13
- net MDO14 renamed MD14
- net MDO15 renamed MD15
- net MDO2 renamed MD2
- net MDO3 renamed MD3
- net MDO4 renamed MD4
- net MDO5 renamed MD5
- net MDO6 renamed MD6
- net MDO7 renamed MD7
- net MDO8 renamed MD8
- net MDO9 renamed MD9
- no-connect marks 7 -> 6
Other:
- note added: "NOTE: Signals drawn backwards on schematic. U9.1 -> U19.2 (blink) U9.2 -> AT7"
- note removed: "BW"
- note removed: "NOTE: hanging line on U9.1"
- moved on the sheet: U2, U26, U27, U38

Commit message: Add files via upload
Other:
- note added: "NOTE: Pin 26 is A13 on the 2764 so you neeed to watch the usage. There was a 2764-based character ROM, but I haven't seen it in the wild. If using a 2764 in place of a 2732 for the regular CGROM, special care is needed."
- note added: "NOTE: The Color Magic uses an Intel D2732A (250nS). The board seems particularly sensitive to what brand/type of 2732 is used, likely due to the access time not being specified on the device. I used a Fujitsu MBM2732A-25 (250nS) which worked fine."
- note removed: "2764A: JP2 - Closed JP3 - Open JP4 - Closed JP5 - Open"
- note removed: "NOTE: The Color Magic uses an Intel D2732A (200nS). The board seems particularly sensitive to what brand/type of 2732 is used (I tried AMD, Fujitsu, and Hitachi with no success). I switched to an AMD2764A and it worked fine."
- moved on the sheet: U15, U2, U27, U3, U4, U50, U9A
