File: Thunder 186/s100_Thunder186-1.0-005.kicad_sch (KiCad schematic)
At the start: 0 parts

Commit message: Add files via upload
Other:
- note added: "NOTES/ERRATA from 1.0-001 to 1.0-002 (not manufactured): 00. 10/15/24 01. Alternative memory arrangement using high-denisity SRAM like the AS6C4008 512kx8-55 configured as 2x128k. NOTES/ERRATA from 1.0-002 to 1.0-003 (manufactured): 00. 10/18/24 01. Changed serial level shifters to higher-density versions; changed serial port headers to accommodate PC motherboard DE9 dongles. NOTES/ERRATA from 1.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"
- note removed: "NOTES/ERRATA from 1.0-001 to 1.0-002 (not manufactured): 01. Alternative memory arrangement using high-denisity SRAM like the AS6C4008 512kx8-55 configured as 2x128k. NOTES/ERRATA from 1.0-002 to 1.0-003 (manufactured): 01. Changed serial level shifters to higher-density versions; changed serial port headers to accommodate PC motherboard DE9 dongles. NOTES/ERRATA from 1.0-003 to 1.0-004 (not manf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"
Changed lines of the file:
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@@
 		)
 	)
-	(text "NOTES/ERRATA from 1.0-001 to 1.0-002 (not manufactured):\n01. Alternative memory arrangement using high-denisity\n    SRAM like the AS6C4008 512kx8-55 configured as\n	2x128k. \n\nNOTES/ERRATA from 1.0-002 to 1.0-003 (manufactured):\n01. Changed serial level shifters to higher-density\n	versions; changed serial port headers to accommodate\n	PC motherboard DE9 dongles.\n\nNOTES/ERRATA from 1.0-003 to 1.0-004 (not manfactured):\n01. U28.7 not connected to J2.7 (bad net name)\n02. Capacitors C3 and C8 are polairty reversed on the\n	79L12 regulator.\n03.	Renamed address bus nets as the internal bus goes\n	right out to the external bus.\n\nNOTES/ERRATA from 1.0-004 to 1.0-005:\n01. Discovered that the footprint for the 80186 was wrong\n	(apparently Intel misnumbered the pins from the standard\n	PLCC68, thus needing a custom footprint).\n\n"
+	(text "NOTES/ERRATA from 1.0-001 to 1.0-002 (not manufactured):\n00. 10/15/24\n01. Alternative memory arrangement using high-denisity\n    SRAM like the AS6C4008 512kx8-55 configured as\n	2x128k. \n\nNOTES/ERRATA from 1.0-002 to 1.0-003 (manufactured):\n00. 10/18/24\n01. Changed serial level shifters to higher-density\n	versions; changed serial port headers to accommodate\n	PC motherboard DE9 dongles.\n\nNOTES/ERRATA from 1.0-003 to 1.0-004 (not manfactured):\n00. 10/18/24. Transient version; not routed.\n01. U28.7 not connected to J2.7 (bad net name)\n02. Capacitors C3 and C8 are polairty reversed on the\n	79L12 regulator.\n03.	Renamed address bus nets as the internal bus goes\n	right out to the external bus.\n\nNOTES/ERRATA from 1.0-004 to 1.0-005:\n00. 11/14/24\n01. Discovered that the footprint for the 80186 was wrong\n	(apparently Intel misnumbered the pins from the standard\n	PLCC68, thus needing a custom footprint).\n\n"
 		(exclude_from_sim no)
 		(at 24.384 140.462 0)
