File: Thunder 186/sch_pg1.kicad_sch (KiCad schematic)
At the start: 23 parts, among them J1 Serial 1, J2 Serial 0, U27 74LS245, U28 MAX1406CPE+, U29 8251A, U30 8251A, U31 MAX1406CPE+, U37 80186-3, U40 27256, U41 27256, U46 74LS06, U49 74LS14, U50 74LS373, U61 74LS14, U72 74LS373, X1 16MHz

Commit message: Add files via upload
Parts:
- removed J1: Serial 1, Connector_PinHeader_2.54mm:PinHeader_2x05_P2.54mm_Vertical, symbol Connector_Generic:Conn_02x05_Odd_Even
- removed J2: Serial 0, Connector_PinHeader_2.54mm:PinHeader_2x05_P2.54mm_Vertical, symbol Connector_Generic:Conn_02x05_Odd_Even
- added J1: Serial 1, Connector_PinHeader_2.54mm:PinHeader_2x10_P2.54mm_Vertical, symbol Connector_Generic:Conn_02x10_Odd_Even
- added J2: Serial 0, Connector_PinHeader_2.54mm:PinHeader_2x10_P2.54mm_Vertical, symbol Connector_Generic:Conn_02x10_Odd_Even
Connections:
- net GND: now also J1.1 (Pin_1), J1.13 (Pin_13), J2.1 (Pin_1), J2.13 (Pin_13)
- net J1_CTS: now also J1.14 (Pin_14)
- net J1_DSR: now also J1.7 (Pin_7)
- net J1_DTR: now also J1.9 (Pin_9)
- net J1_RTS: now also J1.11 (Pin_11)
- net J1_RX: now also J1.3 (Pin_3)
- net J1_TX: now also J1.5 (Pin_5)
- net J2_CTS: now also J2.14 (Pin_14)
- net J2_DSR: now also J2.7 (Pin_7)
- net J2_DTR: now also J2.9 (Pin_9)
- net J2_RTS: now also J2.11 (Pin_11)
- net J2_RX: now also J2.3 (Pin_3)
- net J2_TX: now also J2.5 (Pin_5)
- no-connect marks 24 -> 42
Other:
- note added: "NOTE: J1/J2 connect by a 20-conductor ribbon cable to an IDC DB25F, pin 1 justified."
- note removed: "DCD"
- note removed: "IBM-PC 10-pin Motherboard Connector"
- note removed: "RI"
- moved on the sheet: C37, C38, C39, C40, C41, C42
