File: Thunder 186/sch_pg4.kicad_sch (KiCad schematic)
At the start: 22 parts, among them U33 7406, U36 PAL16L8, U38 74LS245, U39 74LS244, U49 74LS14, U57 74LS04, U58 74LS125, U59 74LS14, U61 74LS14, U62 74LS244, U63 7406, U64 74LS245, U65 74LS244, U66 74LS373, U67 PAL16L8, U68 74LS375, U69 74LS08

Commit message: Add files via upload
Parts:
- removed C9: 2.2u, Capacitor_THT:C_Disc_D4.3mm_W1.9mm_P5.00mm, symbol Device:C
- added C9: 22u, Capacitor_THT:C_Disc_D4.3mm_W1.9mm_P5.00mm, symbol Device:C_Polarized
Connections:
- net GND: now also C9.2
- net at D2.2 (A), R4.1, U61.13: now also C9.1
Changed lines of the file:
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@@
 	(title_block
 		(title "Lomas Thunder 186 Rev. E")
-		(date "2024-11-25")
+		(date "2024-11-28")
 		(rev "1.0-006")
 		(company "Lomas Data Produtcs")
@@
 	)
 	(symbol
+		(lib_id "Device:C_Polarized")
+		(at 55.88 186.69 0)
+		(unit 1)
+		(exclude_from_sim no)
+		(in_bom yes)
+		(on_board yes)
+		(dnp no)
+		(property "Reference" "C9"
+			(at 57.15 184.15 0)
+			(effects
+				(font
+					(size 1.27 1.27)
+				)
+				(justify left)
+			)
+		)
+		(property "Value" "22u"
+			(at 57.15 189.23 0)
+			(effects
+				(font
+					(size 1.27 1.27)
+				)
+				(justify left)
+			)
+		)
+		(property "Footprint" "Capacitor_THT:C_Disc_D4.3mm_W1.9mm_P5.00mm"
+			(at 56.8452 190.5 0)
+			(effects
+				(font
+					(size 1.27 1.27)
+				)
+				(hide yes)
+			)
+		)
+		(property "Datasheet" "~"
+			(at 55.88 186.69 0)
+			(effects
+				(font
+					(size 1.27 1.27)
+				)
+				(hide yes)
+			)
+		)
+		(property "Description" ""
+			(at 55.88 186.69 0)
+			(effects
+				(font
+					(size 1.27 1.27)
+				)
+				(hide yes)
+			)
+		)
+		(pin "1"
+		)
+		(pin "2"
+		)
+		(instances
+			(project "s100_Thunder186-1.0-006"
+				(path "/048cf1fc-81fe-43c0-b445-36f3c2f214da/f18f69ea-453b-4e6e-a333-4a79be0636c4"
+					(reference "C9")
+					(unit 1)
+				)
+			)
+		)
+	)
+	(symbol
 		(lib_id "74xx:74LS14")
 		(at 359.41 152.4 180)
@@
 				)
 			)
-		)
-	)
-	(symbol
-		(lib_id "Device:C")
-		(at 55.88 186.69 0)
-		(unit 1)
-		(exclude_from_sim no)
-		(in_bom yes)
-		(on_board yes)
-		(dnp no)
-		(property "Reference" "C9"
-			(at 57.15 184.15 0)
-			(effects
-				(font
-					(size 1.27 1.27)
-				)
-				(justify left)
-			)
-		)
-		(property "Value" "2.2u"
-			(at 57.15 189.23 0)
-			(effects
-				(font
-					(size 1.27 1.27)
-				)
-				(justify left)
-			)
-		)
-		(property "Footprint" "Capacitor_THT:C_Disc_D4.3mm_W1.9mm_P5.00mm"
-			(at 56.8452 190.5 0)
-			(effects
-				(font
-					(size 1.27 1.27)
-				)
-				(hide yes)
-			)
-		)
-		(property "Datasheet" "~"
-			(at 55.88 186.69 0)
-			(effects
-				(font
-					(size 1.27 1.27)
-				)
-				(hide yes)
-			)
-		)
-		(property "Description" ""
-			(at 55.88 186.69 0)
-			(effects
-				(font
-					(size 1.27 1.27)
-				)
-				(hide yes)
-			)
-		)
-		(pin "1"
-		)
-		(pin "2"
-		)
-		(instances
-			(project "s100_Thunder186-1.0-001"
-				(path "/048cf1fc-81fe-43c0-b445-36f3c2f214da/f18f69ea-453b-4e6e-a333-4a79be0636c4"
-					(reference "C9")
-					(unit 1)
-				)
-			)

Commit message: Add files via upload
Parts:
- C9: footprint Capacitor_THT:C_Disc_D4.3mm_W1.9mm_P5.00mm -> Capacitor_THT:CP_Radial_Tantal_D4.5mm_P2.50mm
Other:
- note added: "NOTE: R4 is 5.1k on the schematic and C9 is drawn as a non-polarized cap."
- note removed: "NOTE: R4 is 5.1k on the schematic."
Changed lines of the file:
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@@
 	(title_block
 		(title "Lomas Thunder 186 Rev. E")
-		(date "2024-11-28")
+		(date "2024-12-01")
 		(rev "1.0-006")
 		(company "Lomas Data Produtcs")
@@
 		)
 	)
-	(text "NOTE: R4 is 5.1k on the schematic."
+	(text "NOTE: R4 is 5.1k on the schematic and C9 is\ndrawn as a non-polarized cap."
 		(exclude_from_sim no)
 		(at 57.15 199.644 0)
@@
 			)
 		)
-		(property "Footprint" "Capacitor_THT:C_Disc_D4.3mm_W1.9mm_P5.00mm"
+		(property "Footprint" "Capacitor_THT:CP_Radial_Tantal_D4.5mm_P2.50mm"
 			(at 56.8452 190.5 0)
 			(effects
